File: pcb/vabo-rev01/openX65-vabo.kicad_pcb (KiCad board)
At the start: 2 copper layers, 100 x 100 mm, 190 parts, among them J302 S-video, J303 VGA, J401 SD_Card_wSwitches, J501 SOCK 2x10p 2,54mm, J502 SOCK 2x10p 2,54mm, J701 Lumberg 1503-07, J702 PINS 1x2, J703 PINS 1x2, J801 RJ45_Amphenol_RJMG1BD3B8K1ANR, Q201 BSS123, Q701 BSS123, SW701 5MS3S102AM6QE, U201 ICE40UP5K-SG48ITR50, U301 THS7314D, U401 W25Q16JVSNIQ, U402 74CBTLV3126PW,118, U403 74AHC00PW, U404 74CBTLV3126PW,118, U501 74LVC1G11, U601 ICE5LP1K-SG48, U602 74CBTLV3126PW,118, U603 W25Q16JVSNIQ, U701 WM8524CGEDT, U702 LM4890MX, U801 W6100L, X201 SG5032CAN_25.000000M-TJGA3, Y801 ABM3-25.000MHZ-D2Y-T

Commit message: V/A board rev01 finished and submitted to pcbway
Parts:
- removed C204, C301, C605: 1u, Capacitor_SMD:C_0603_1608Metric_Pad1.08x0.95mm_HandSolder
- removed FID104: Fiducial, Fiducial:Fiducial_1mm_Mask2mm
- removed JP401: Flash enable, Connector_PinHeader_2.54mm:PinHeader_1x02_P2.54mm_Vertical
- removed R805: 10k, Resistor_SMD:R_0603_1608Metric_Pad0.98x0.95mm_HandSolder
- added C501: 1u, Capacitor_SMD:C_0603_1608Metric_Pad1.08x0.95mm_HandSolder, F.Cu at (96.5, 135.6)
- added C502: 22u/16V, Capacitor_SMD:C_0805_2012Metric_Pad1.18x1.45mm_HandSolder, F.Cu at (98.6, 75.0)
- added C712: 3u3, Capacitor_SMD:C_0603_1608Metric_Pad1.08x0.95mm_HandSolder, F.Cu at (96.5, 46.5)
- added C713: 1u, Capacitor_SMD:C_0603_1608Metric_Pad1.08x0.95mm_HandSolder, F.Cu at (108.8, 47.2)
- added C714: 1uF, Capacitor_SMD:C_0603_1608Metric_Pad1.08x0.95mm_HandSolder, F.Cu at (110.5, 47.2)
- added C715: 2n7, Capacitor_SMD:C_0603_1608Metric_Pad1.08x0.95mm_HandSolder, F.Cu at (102.2, 50.4)
- added C716: 2n7, Capacitor_SMD:C_0603_1608Metric_Pad1.08x0.95mm_HandSolder, F.Cu at (94.5, 49.0)
- added C717: 4u7, Capacitor_SMD:C_0603_1608Metric_Pad1.08x0.95mm_HandSolder, F.Cu at (98.5, 46.5)
- added C718: 4u7, Capacitor_SMD:C_0603_1608Metric_Pad1.08x0.95mm_HandSolder, F.Cu at (109.8, 50.4)
- added C719: 22u/16V, Capacitor_SMD:C_0805_2012Metric_Pad1.18x1.45mm_HandSolder, F.Cu at (72.4, 47.7)
- added C816: 22u/16V, Capacitor_SMD:C_0805_2012Metric_Pad1.18x1.45mm_HandSolder, F.Cu at (131.7, 127.8)
- added C817: 22u/16V, Capacitor_SMD:C_0805_2012Metric_Pad1.18x1.45mm_HandSolder, F.Cu at (105.0, 103.5)
- added C818: 1nF/2kV, Capacitor_SMD:C_1206_3216Metric_Pad1.33x1.80mm_HandSolder, F.Cu at (147.4, 131.2)
- added D501: AA4040LCGCK-AMT, ledplcc2:PLCC2_4x4mm, F.Cu at (62.4, 70.8)
- added D502: AA4040SESK, ledplcc2:PLCC2_4x4mm, F.Cu at (62.4, 109.7)
- added D503: AA4040SESK, ledplcc2:PLCC2_4x4mm, F.Cu at (62.4, 116.2)
- added D605: LED_GREEN_0603, LED_SMD:LED_0603_1608Metric_Pad1.05x0.95mm_HandSolder, F.Cu at (87.9, 43.6)
- added J301: Composite, Connector_PinHeader_2.54mm:PinHeader_1x02_P2.54mm_Vertical, F.Cu at (145.3, 63.3)
- added J503: Conn_01x01, Connector_PinHeader_2.54mm:PinHeader_1x01_P2.54mm_Vertical, F.Cu at (76.0, 66.9)
- added J504: Conn_01x01, Connector_PinHeader_2.54mm:PinHeader_1x01_P2.54mm_Vertical, F.Cu at (142.2, 78.6)
- added Q401: BSS138, Package_TO_SOT_SMD:SOT-23, F.Cu at (68.2, 118.0)
- added Q601: BSS138, Package_TO_SOT_SMD:SOT-23, F.Cu at (84.2, 44.8)
- added R323: 27R, Resistor_SMD:R_0603_1608Metric_Pad0.98x0.95mm_HandSolder, F.Cu at (140.5, 81.5)
- added R324: 160R, Resistor_SMD:R_0603_1608Metric_Pad0.98x0.95mm_HandSolder, F.Cu at (140.5, 83.3)
- added R325: 150R, Resistor_SMD:R_0603_1608Metric_Pad0.98x0.95mm_HandSolder, F.Cu at (140.6, 85.1)
- added R326: 27R, Resistor_SMD:R_0603_1608Metric_Pad0.98x0.95mm_HandSolder, F.Cu at (140.6, 88.9)
- added R327: 160R, Resistor_SMD:R_0603_1608Metric_Pad0.98x0.95mm_HandSolder, F.Cu at (140.6, 90.7)
- added R328: 150R, Resistor_SMD:R_0603_1608Metric_Pad0.98x0.95mm_HandSolder, F.Cu at (140.6, 92.5)
- added R329: 27R, Resistor_SMD:R_0603_1608Metric_Pad0.98x0.95mm_HandSolder, F.Cu at (140.7, 96.0)
- added R330: 160R, Resistor_SMD:R_0603_1608Metric_Pad0.98x0.95mm_HandSolder, F.Cu at (140.7, 99.6)
- added R331: 150R, Resistor_SMD:R_0603_1608Metric_Pad0.98x0.95mm_HandSolder, F.Cu at (140.7, 97.8)
- added R413: 4k7, Resistor_SMD:R_0603_1608Metric_Pad0.98x0.95mm_HandSolder, F.Cu at (95.7, 67.2)
- added R414: 4k7, Resistor_SMD:R_0603_1608Metric_Pad0.98x0.95mm_HandSolder, F.Cu at (89.7, 74.4)
- added R507: 470R, Resistor_SMD:R_0603_1608Metric_Pad0.98x0.95mm_HandSolder, F.Cu at (66.9, 67.5)
- added R508: 470R, Resistor_SMD:R_0603_1608Metric_Pad0.98x0.95mm_HandSolder, F.Cu at (66.8, 107.8)
- added R509: 470R, Resistor_SMD:R_0603_1608Metric_Pad0.98x0.95mm_HandSolder, F.Cu at (67.4, 114.2)
- added R510: 10k, Resistor_SMD:R_0603_1608Metric_Pad0.98x0.95mm_HandSolder, F.Cu at (83.8, 134.0)
- added R511: 10k, Resistor_SMD:R_0603_1608Metric_Pad0.98x0.95mm_HandSolder, F.Cu at (83.7, 131.5)
- added R514: 0R, Resistor_SMD:R_0603_1608Metric_Pad0.98x0.95mm_HandSolder, F.Cu at (106.1, 72.9)
- added R619: 470R, Resistor_SMD:R_0603_1608Metric_Pad0.98x0.95mm_HandSolder, F.Cu at (88.0, 45.3)
- added R709: 560R, Resistor_SMD:R_0603_1608Metric_Pad0.98x0.95mm_HandSolder, F.Cu at (145.0, 55.1)
- added R710: 560R, Resistor_SMD:R_0603_1608Metric_Pad0.98x0.95mm_HandSolder, F.Cu at (143.1, 50.1)
- added R712: 560R, Resistor_SMD:R_0603_1608Metric_Pad0.98x0.95mm_HandSolder, F.Cu at (106.0, 50.1)
- added R713: 560R, Resistor_SMD:R_0603_1608Metric_Pad0.98x0.95mm_HandSolder, F.Cu at (97.5, 50.1)
- added SW401: PTS645VM13SMTR92 LFS, switches:PTS645VM13SMTR92 LFS, F.Cu at (60.4, 126.0)
- added SW501: A6SN-4101, Button_Switch_SMD:SW_DIP_SPSTx04_Slide_Omron_A6S-410x_W8.9mm_P2.54mm, F.Cu at (76.1, 130.1)
- added U502: 74LVC1G11, Package_TO_SOT_SMD:SOT-23-6_Handsoldering, F.Cu at (88.0, 51.1)
- added U503: 74LVC2G02, Package_SO:TSSOP-8_3x3mm_P0.65mm, F.Cu at (99.2, 132.3)
- added U504: 74CBTLV3126PW,118, Package_SO:TSSOP-14_4.4x5mm_P0.65mm, F.Cu at (90.5, 131.2)
- added U505: 74AHCT573PW, Package_SO:TSSOP-20_4.4x6.5mm_P0.65mm, F.Cu at (95.7, 123.1)
- added U703: WM8524CGEDT, Package_SO:TSSOP-16_4.4x5mm_P0.65mm, F.Cu at (103.7, 46.6)
- C302: value 10uF -> 22u/16V
- C701: value 2.2uF -> 3u3
- C703, C709, C711: value 1uF -> 1u
- C704, C705: value 2.7nF -> 2n7
- C706, C707: value 4.7uF -> 4u7
- D203: value LTST-S270GKT -> LED_GREEN_0603
- J302: value S-video -> DS1093-01-BN40; footprint vera-module:MD-40S -> vera-module:DS1093-01-BN40
- J303: value VGA -> ICD15S13E4GV00LF
- J401: value SD_Card_wSwitches -> DM1AA-SF-PEJ
- J801: value RJ45_Amphenol_RJMG1BD3B8K1ANR -> RJMG1BD3B8K1ANR
- JP402: moved to B.Cu
- Q201, Q701: value BSS123 -> BSS138
- R303, R304: value 470 -> 470R
- R305: value 0 -> 0R
- R306, R307, R308: value 75 -> 75R
- R309, R313, R317: value 536 -> 510R
- R310, R314, R318: value 1070 -> 910R
- R311, R315, R319: value 2150 -> 2k
- R312, R316, R320: value 4300 -> 4k3
- R321, R322: value 820 -> 820R
- R701, R702: value 560 -> 560R
- R804: value 10k -> 10M; footprint Resistor_SMD:R_0603_1608Metric_Pad0.98x0.95mm_HandSolder -> Resistor_SMD:R_2512_6332Metric_Pad1.40x3.35mm_HandSolder
- U601: value ICE5LP1K-SG48 -> ICE5LP{1,2,4}K-SG48
- moved R201 127.7 mm to (133.7, 50.6), turned to -90 degrees
- moved R203 126.1 mm to (83.7, 48.4)
- moved R501 122.7 mm to (104.0, 86.5), turned to -90 degrees
- moved R207 120.6 mm to (76.3, 45.8), turned to 180 degrees
- moved R502 119.2 mm to (107.0, 67.3), turned to 180 degrees
- moved U501 119.2 mm to (116.9, 50.6)
- moved R605 116.7 mm to (102.9, 57.6)
- moved D203 116.4 mm to (76.3, 43.7)
- moved Q201 112.2 mm to (80.4, 44.9), turned to 90 degrees
- moved R505 112.1 mm to (110.4, 67.3)
- moved C603 110.0 mm to (104.0, 76.9), turned to 180 degrees
- moved FB804 109.9 mm to (106.9, 108.1), turned to 90 degrees
- moved C608 109.7 mm to (110.6, 70.5), turned to 90 degrees
- moved C606 109.0 mm to (103.2, 79.7), turned to -90 degrees
- moved R410 108.9 mm to (88.8, 108.8), turned to -90 degrees
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Connections:
- net Net-(C710-Pad1) renamed /Audio DAC, Output/AMPINN
- net Net-(C710-Pad2) renamed /Audio DAC, Output/SPK1
- net Net-(C808-Pad1) renamed /Ethernet/3V3D
- net Net-(C810-Pad2) renamed /Ethernet/CTVDD
- net Net-(C813-Pad1) renamed /Ethernet/XSCO
- net Net-(C814-Pad1) renamed /Ethernet/XSCI
- net Net-(C815-Pad2) renamed /Ethernet/~{WIZRST}
- net Net-(J303-Pad13) renamed /Video Outputs/HSYNC
- net Net-(J303-Pad14) renamed /Video Outputs/VSYNC
- net Net-(J401-Pad1) renamed /VERA SPI-Flash, SDC/CDDAT3
- net Net-(J401-Pad2) renamed /VERA SPI-Flash, SDC/CMD
- net Net-(J401-Pad5) renamed /VERA SPI-Flash, SDC/CLK
- net Net-(J401-Pad7) renamed /VERA SPI-Flash, SDC/DAT0
- net Net-(J401-Pad8) renamed /VERA SPI-Flash, SDC/DAT1
- net Net-(J401-Pad9) renamed /VERA SPI-Flash, SDC/DAT2
- net Net-(J702-Pad2) renamed /Audio DAC, Output/SPK2
- net Net-(J801-PadL2) renamed /Ethernet/LEDYK
- net Net-(J801-PadL3) renamed /Ethernet/LEDGK
- net Net-(R201-Pad2) renamed /Video VERA FPGA/VFPGA_CRESB
- net Net-(R204-Pad1) renamed /Video VERA FPGA/25MHZ
- net Net-(R604-Pad2) renamed /Audio AURA FPGA/AFRESB
- net Net-(R701-Pad2) renamed /Audio DAC, Output/LINEOUTL
- net Net-(R702-Pad2) renamed /Audio DAC, Output/LINEOUTR
- net Net-(R801-Pad1) renamed /Ethernet/RSET
- net Net-(R803-Pad1) renamed /Ethernet/MOD0
- net Net-(R806-Pad2) renamed /Ethernet/MOD2
- net Net-(R807-Pad1) renamed /Ethernet/~{LLED}
- net Net-(R808-Pad1) renamed /Ethernet/~{ALED}
- net Net-(U601-Pad7) renamed AFPGA_CDONE
- J303 pad 1: Net-(J303-Pad1) -> /Video Outputs/RED
- J303 pad 2: Net-(J303-Pad2) -> /Video Outputs/GREEN
- J303 pad 3: Net-(J303-Pad3) -> /Video Outputs/BLUE
- J502 pad 1: VAUX1 -> NAUDIO_BCK
- J502 pad 13: FCDONE -> /Motherboard Connectors/FCDONE
- J502 pad 4: ~{ERST} -> NAUDIO_DATA
- J502 pad 6: VAUX2 -> NAUDIO_LRCK
- J701 pad R: unconnected-(J701-PadR) -> /Audio DAC, Output/RJACK
- J701 pad S: unconnected-(J701-PadS) -> GND
- J701 pad T: unconnected-(J701-PadT) -> /Audio DAC, Output/LJACK
- J801 pad 13: unconnected-(J801-Pad13) -> /Ethernet/LANSH
- R309 pad 1: Net-(J303-Pad1) -> Net-(R309-Pad1)
- R310 pad 1: Net-(J303-Pad1) -> Net-(R310-Pad1)
- R311 pad 1: Net-(J303-Pad1) -> Net-(R311-Pad1)
- R312 pad 1: Net-(J303-Pad1) -> /Video Outputs/RED
- R313 pad 1: Net-(J303-Pad2) -> Net-(R313-Pad1)
- R314 pad 1: Net-(J303-Pad2) -> Net-(R314-Pad1)
- R315 pad 1: Net-(J303-Pad2) -> Net-(R315-Pad1)
- R316 pad 1: Net-(J303-Pad2) -> /Video Outputs/GREEN
- R317 pad 1: Net-(J303-Pad3) -> Net-(R317-Pad1)
- R318 pad 1: Net-(J303-Pad3) -> Net-(R318-Pad1)
- R319 pad 1: Net-(J303-Pad3) -> Net-(R319-Pad1)
- R320 pad 1: Net-(J303-Pad3) -> /Video Outputs/BLUE
- R804 pad 1: Net-(R804-Pad1) -> /Ethernet/LANSH
- U403 pad 12: VFPGA_CDONE -> Net-(U403-Pad10)
- U403 pad 13: Net-(U403-Pad10) -> VFPGA_CDONE
- U404 pad 11: FMISO -> FMOSI
- U404 pad 12: VSPI_MISO -> VSPI_MOSI
- U404 pad 5: VSPI_MOSI -> VSPI_MISO
- U404 pad 6: FMOSI -> FMISO
- U601 pad 10: ~{MWR} -> VAUDIO_DATA
- U601 pad 11: ~{VCS0} -> VAUDIO_BCK
- U601 pad 12: ~{ACS1} -> AUDIO_BCK
- U601 pad 13: unconnected-(U601-Pad13) -> AUDIO_DATA
- U601 pad 18: D7 -> AUDIO_LRCK
- U601 pad 19: D6 -> unconnected-(U601-Pad19)
- U601 pad 2: AUDIO_LRCK -> D7
- U601 pad 20: D5 -> unconnected-(U601-Pad20)
- U601 pad 21: D4 -> unconnected-(U601-Pad21)
- U601 pad 23: D3 -> unconnected-(U601-Pad23)
- U601 pad 25: D2 -> ~{AIRQ}
- U601 pad 26: D1 -> ~{ACS1}
- U601 pad 27: D0 -> ~{IOCS}
- U601 pad 28: A0 -> ~{VCS0}
- U601 pad 3: ~{SD_CD} -> unconnected-(U601-Pad3)
- U601 pad 31: A1 -> unconnected-(U601-Pad31)
- U601 pad 32: A2 -> D0
- U601 pad 34: A3 -> A4
- U601 pad 36: A4 -> ~{MRD}
- U601 pad 37: A5 -> A2
- U601 pad 38: A6 -> A3
- U601 pad 39: unconnected-(U601-Pad39) -> A1
- U601 pad 4: SD_WP -> unconnected-(U601-Pad4)
- U601 pad 40: unconnected-(U601-Pad40) -> A0
- U601 pad 42: A7 -> ~{MWR}
- U601 pad 43: unconnected-(U601-Pad43) -> D1
- U601 pad 44: VAUDIO_LRCK -> D2
- U601 pad 45: AUDIO_DATA -> D3
- U601 pad 46: VAUDIO_BCK -> D4
- U601 pad 47: VAUDIO_DATA -> D5
- U601 pad 48: AUDIO_BCK -> D6
- U601 pad 6: ~{AIRQ} -> unconnected-(U601-Pad6)
- U601 pad 9: ~{MRD} -> VAUDIO_LRCK
- U801 pad 26: Net-(R804-Pad1) -> GND
- U801 pad 28: Net-(R805-Pad1) -> GND
Routing:
- net GND: track 0.00 -> 1446.7 mm, vias 0 -> 133
- net +3V3: track 0.00 -> 816.7 mm, vias 0 -> 42
- net VFPGA_CDONE: track 0.00 -> 208.4 mm, vias 0 -> 10
- net ~{EIRQ}: track 0.00 -> 177.4 mm, vias 0 -> 5
- net ~{ECS2}: track 0.00 -> 158.5 mm, vias 0 -> 3
- net +1V2: track 0.00 -> 150.4 mm, vias 0 -> 9
- net ~{VSPI_SSEL}: track 0.00 -> 142.4 mm, vias 0 -> 8
- net ASYSCLK: track 0.00 -> 141.9 mm, vias 0 -> 11
- net ~{MRD}: track 0.00 -> 130.5 mm, vias 0 -> 3
- net D0: track 0.00 -> 116.4 mm, vias 0 -> 4
- net D1: track 0.00 -> 106.5 mm, vias 0 -> 4
- net +5V: track 0.00 -> 105.3 mm, vias 0 -> 3
- net D2: track 0.00 -> 104.3 mm, vias 0 -> 4
- net D3: track 0.00 -> 104.0 mm, vias 0 -> 4
- net A1: track 0.00 -> 98.5 mm, vias 0 -> 4
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- added copper zone on B.Cu, net GND
- added copper zone on F.Cu, net GND
Other:
- board text added: "1"
- board text added: "2"
- board text added: "3"
- board text added: "4"
- board text added: "AURA"
- board text added: "Composite pin-header"
- board text added: "GND"
- board text added: "LAN"
- board text added: "LAN 10/100 (top side)"
- board text added: "LOUD"
- board text added: "Line Audio Out (top side)"
- board text added: "MEET US AT X65.EU"
- board text added: "MUTE"
- board text added: "OpenX65 V/A-bo rev01"
- board text added: "QUIET"
- board text added: "S-Video out (top side)"
- board text added: "Speaker Volume (top side)"
- board text added: "VERA"
- board text added: "VERA (READY) AURA"
- board text added: "VGA Output (top side)"
- board text added: "X65.EU"
