File: pcb/vabo-rev01/openX65-vabo.kicad_sch (KiCad schematic)
At the start: 8 parts

Commit message: V/A board rev01 finished and submitted to pcbway
Parts:
- removed FID104: Fiducial, Fiducial:Fiducial_1mm_Mask2mm, symbol Mechanical:Fiducial
- FID101, FID102, FID103, H101, H102, H103, H104: now left out of the parts list
Other:
- sheet VERA SPI-Flash, SDHC renamed VERA SPI-Flash, SDC
- note added: "2"
- note added: "3"
- note added: "4"
- note added: "5"
- note added: "6"
- note added: "7"
- note added: "8"
- note added: "8-bit bus"
- note added: "AURA FPGA"
- note added: "Amp."
- note added: "Audio Line output"
- note added: "Block Diagram:"
- note added: "DAC"
- note added: "DAC (opt.)"
- note added: "Description"
- note added: "Initial design, PCB 100x100mm 2-layers. VERA with VGA and S-Video outputs. AURA with line-out and amp/speaker, 2 DAC. LAN by W6100L"
- note added: "Motherboard Connectors Two 2x10p 2.54mm headers"
- note added: "OpenX65 Video/Audio & Ethernet Board ("V/A-BO")"
- note added: "RJ45 for 10/100 Ethernet"
- note added: "Rev. / Date"
- note added: "Revision History:"
- note added: "S-Video output VGA output"
- note added: "SD-Card slot"
- note added: "Sheet 2, 3, 4"
- note added: "Sheet 6"
- note added: "Sheet 7"
- note added: "Sheet 8"
- note added: "Sheets:"
- note added: "Sound from VERA"
- note added: "Speaker mono"
- note added: "VERA FPGA"
- note added: "W6100L LAN"
- note added: "rev01 / 28.4.2023"
- note removed: "OpenX65 Video/Audio & Ethernet Board ("VABO")"
- company: (none) -> FOR X65.EU DESIGNED BY JSYKORA.INFO
- title: (none) -> OpenX65 - Video/Audio & Ethernet Board
- moved on the sheet: FID101, FID102, FID103, H101, H102, H103, H104
