File: pcb/vabo-rev01/vabo-sheet-02.kicad_sch (KiCad schematic)
At the start: 19 parts, among them Q201 BSS138, U201 ICE40UP5K-SG48ITR50, X201 SG5032CAN_25.000000M-TJGA3

Commit message: V/A board rev01 finished and submitted to pcbway
Parts:
- removed C204: 1u, Capacitor_SMD:C_0603_1608Metric_Pad1.08x0.95mm_HandSolder, symbol Device:C_Small
- D203: value LTST-S270GKT -> LED_GREEN_0603
Connections:
- net 25MHZ: now reaches R204.1, R205.1, R206.1, X201.3 (OUT)
- net VFPGA_CRESB: now reaches R201.2, R208.2, U201.8 (CRESET_B)
Other:
- note added: ""VERA READY" internal LED"
- note added: "package QFN-48"
- note removed: ""VERA READY""
- note removed: "TBD: LED footprint"
- company: (none) -> FOR X65.EU DESIGNED BY JSYKORA.INFO
- title: (none) -> OpenX65 - Video/Audio & Ethernet Board
- moved on the sheet: R201, R208
