File: pcb/vabo-rev01/vabo-sheet-03.kicad_sch (KiCad schematic)
At the start: 38 parts, among them J301 Composite, J302 S-video, J303 VGA, U301 THS7314D

Commit message: V/A board rev01 finished and submitted to pcbway
Parts:
- removed C301: 1u, Capacitor_SMD:C_0603_1608Metric_Pad1.08x0.95mm_HandSolder, symbol Device:C_Small
- added R323, R326, R329: 27R, Resistor_SMD:R_0603_1608Metric_Pad0.98x0.95mm_HandSolder, symbol Device:R_Small
- added R324, R327, R330: 160R, Resistor_SMD:R_0603_1608Metric_Pad0.98x0.95mm_HandSolder, symbol Device:R_Small
- added R325, R328, R331: 150R, Resistor_SMD:R_0603_1608Metric_Pad0.98x0.95mm_HandSolder, symbol Device:R_Small
- C302: value 10uF -> 22u/16V
- J301: footprint vera-module:RCJ-014 -> Connector_PinHeader_2.54mm:PinHeader_1x02_P2.54mm_Vertical
- J302: value S-video -> DS1093-01-BN40; footprint vera-module:MD-40S -> vera-module:DS1093-01-BN40; symbol Connector:Mini-DIN-4 -> vera-module:Mini-DIN-4-SH
- J303: value VGA -> ICD15S13E4GV00LF
- R303, R304: value 470 -> 470R
- R305: value 0 -> 0R
- R306, R307, R308: value 75 -> 75R
- R309, R313, R317: value 536 -> 510R
- R310, R314, R318: value 1070 -> 910R
- R311, R315, R319: value 2150 -> 2k
- R312, R316, R320: value 4300 -> 4k3
- R321, R322: value 820 -> 820R
Connections:
- net GND: now also J302.SH
- net VSYNC: now reaches J303.14, R321.1
- net HSYNC: now reaches J303.13, R322.1
- new net: R311.1, R325.2
- new net: R314.1, R327.2
- new net: R313.1, R326.2
- new net: R318.1, R330.2
- new net: R310.1, R324.2
- new net: R315.1, R328.2
- new net: R309.1, R323.2
- new net: R319.1, R331.2
- new net: R317.1, R329.2
- new net BLUE: J303.3, R320.1, R329.1, R330.1, R331.1
- new net GREEN: J303.2, R316.1, R326.1, R327.1, R328.1
- new net RED: J303.1, R312.1, R323.1, R324.1, R325.1
Other:
- note added: "(orig: 536R)"
- note added: "(orig:536R)"
- note added: "Due to lack of PCB space, the J301 is implemented as a pin-header only."
- note added: "S-Video Output"
- note added: "package: SOIC-8, 3.9x4.9mm"
- note removed: "Due to lack of PCB space, the J301 is not in PCB."
- note removed: "TBD: check if resistors in series!!"
- note removed: "https://www.qsl.net/in3otd/parallr.html#"
- company: (none) -> FOR X65.EU DESIGNED BY JSYKORA.INFO
- title: (none) -> OpenX65 - Video/Audio & Ethernet Board
- moved on the sheet: C302, R305, R309, R310, R311, R312, R313, R314, R315, R316, R317, R318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
