File: pcb/vabo-rev01/vabo-sheet-04.kicad_sch (KiCad schematic)
At the start: 27 parts, among them J401 DM1AA-SF-PEJ, SW401 SW_Push, U401 W25Q16JVSNIQ, U402 74CBTLV3126PW,118, U403 74AHC00PW, U404 74CBTLV3126PW,118

Commit message: V/A board rev01 finished and submitted to pcbway
Parts:
- removed D401: CUS10S30,H3F, Diode_SMD:D_SOD-323_HandSoldering, symbol Device:D_Schottky
- removed JP401: Flash enable, Connector_PinHeader_2.54mm:PinHeader_1x02_P2.54mm_Vertical, symbol Jumper:Jumper_2_Open
- added Q401: BSS138, Package_TO_SOT_SMD:SOT-23, symbol Transistor_FET:BSS123
- added R414: 4k7, Resistor_SMD:R_0603_1608Metric_Pad0.98x0.95mm_HandSolder, symbol Device:R
- JP402: now left out of the parts list
- SW401: value SW_Push -> PTS645VM13SMTR92 LFS; footprint (none) -> switches:PTS645VM13SMTR92 LFS; symbol Switch:SW_Push -> vera-module:SW_Push_SH
Connections:
- net FMISO: now also U404.6 (2B); no longer U404.11 (4B)
- net FMOSI: now also U404.11 (4B); no longer U404.6 (2B)
- net GND: now also SW401.SH, Q401.2 (S)
- net VFPGA_CDONE: now also U403.13; no longer U403.12
- net VSPI_MISO: now also U404.5 (2A); no longer U404.12 (4A)
- net VSPI_MOSI: now also U404.12 (4A), R414.1; no longer U404.5 (2A)
- net ~{VSPI_SSEL}: now also Q401.1 (G)
- net CMD: now reaches J401.2 (CMD), R404.2, U402.6 (2B)
- net DAT0: now reaches J401.7 (DAT0), R403.2, U402.11 (4B)
- net CDDAT3: now reaches J401.1 (CD/DAT3), R405.2, U402.3 (1B)
- net CLK: now reaches J401.5 (CLK), R406.1, U402.8 (3B)
- net DAT2: now reaches J401.9 (DAT2), R408.2
- net BTNH: now reaches R413.2, SW401.1
- net BTNH: now also R414.2
- net DAT1: now reaches J401.8 (DAT1), R407.2
- net BTNL: now reaches SW401.2
- net BTNL: now also Q401.3 (D)
- net VSPI_SSEL: no longer names the net of U403.10, U403.6
- net VSPI_SSEL: now also U403.12; no longer U403.13
Other:
- note added: "Secure Digital Interface - like an "FDD""
- note added: "VERA push-button Piggy-back on MISO line"
- note added: "dnp"
- note added: "package TSSOP-14 4.4x5mm"
- note added: "package: SOIC-8 3.9x4.9mm"
- note removed: "Secure Digital Interface - "FDD" Concept"
- company: (none) -> FOR X65.EU DESIGNED BY JSYKORA.INFO
- title: (none) -> OpenX65 - Video/Audio & Ethernet Board
- moved on the sheet: C401, C402, C403, J401, R401, R402, R403, R404, R405, R406, R407, R408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
