File: pcb/vabo-rev01/vabo-sheet-05.kicad_sch (KiCad schematic)
At the start: 9 parts, among them J501 SOCK 2x10p 2,54mm, J502 SOCK 2x10p 2,54mm, U501 74LVC1G11

Commit message: V/A board rev01 finished and submitted to pcbway
Parts:
- added C501: 1u, Capacitor_SMD:C_0603_1608Metric_Pad1.08x0.95mm_HandSolder, symbol Device:C_Small
- added C502: 22u/16V, Capacitor_SMD:C_0805_2012Metric_Pad1.18x1.45mm_HandSolder, symbol Device:C
- added D501: AA4040LCGCK-AMT, ledplcc2:PLCC2_4x4mm, symbol Device:LED
- added D502, D503: AA4040SESK, ledplcc2:PLCC2_4x4mm, symbol Device:LED
- added J503, J504: Conn_01x01, Connector_PinHeader_2.54mm:PinHeader_1x01_P2.54mm_Vertical, symbol Connector_Generic:Conn_01x01
- added R507, R508, R509: 470R, Resistor_SMD:R_0603_1608Metric_Pad0.98x0.95mm_HandSolder, symbol Device:R
- added R510, R511: 10k, Resistor_SMD:R_0603_1608Metric_Pad0.98x0.95mm_HandSolder, symbol Device:R
- added R514: 0R, Resistor_SMD:R_0603_1608Metric_Pad0.98x0.95mm_HandSolder, symbol Device:R
- added SW501: A6SN-4101, Button_Switch_SMD:SW_DIP_SPSTx04_Slide_Omron_A6S-410x_W8.9mm_P2.54mm, symbol Switch:SW_DIP_x04
- added U502: 74LVC1G11, Package_TO_SOT_SMD:SOT-23-6_Handsoldering, symbol 74xGxx:74LVC1G11
- added U503: 74LVC2G02, Package_SO:TSSOP-8_3x3mm_P0.65mm, symbol 74xGxx:74LVC2G02
- added U504: 74CBTLV3126PW,118, Package_SO:TSSOP-14_4.4x5mm_P0.65mm, symbol vera-module:74CBTLV3126PW,118
- added U505: 74AHCT573PW, Package_SO:TSSOP-20_4.4x6.5mm_P0.65mm, symbol Logic574:74AHCT573PW
Connections:
- net +1V2: now also C502.2
- net +3V3: now also C501.1, D501.2 (A), D502.2 (A), D503.2 (A), R510.2, R511.2, U502.5 (VCC), U503.8 (VCC), U503.8 (VCC), U504.14 (VCC), U505.20 (VCC)
- net AFPGA_CDONE: now also U502.6
- net D0: now also U504.2 (1A), U505.5 (D3)
- net D1: now also U504.5 (2A), U505.4 (D2)
- net D2: now also U504.12 (4A), U505.3 (D1)
- net D3: now also U504.9 (3A), U505.2 (D0)
- net FCDONE: now also U502.4
- net GND: now also C501.2, C502.1, J503.1 (Pin_1), J504.1 (Pin_1), SW501.5, SW501.6, SW501.7, SW501.8, U502.2 (GND), U503.4 (GND), U503.4 (GND), U504.7 (GND), U505.1 (~{OE}), U505.10 (GND), U505.6 (D4), U505.7 (D5), U505.8 (D6), U505.9 (D7)
- net VFPGA_CDONE: now also SW501.3, U502.1, U502.3
- net ~{ACS1}: now also R514.1
- net ~{ERST}: now also U505.19 (Q0); no longer J502.4 (Pin_4)
- net ~{MRD}: now also U503.5
- net ~{MWR}: now also U503.1
- net VAUX1 renamed NAUDIO_BCK
- net VAUX2 renamed NAUDIO_LRCK
- new net: D502.1 (K), R508.1
- new net: D503.1 (K), R509.1
- new net: D501.1 (K), R507.1
- new net DIP1: R510.1, SW501.1, U504.8 (3B)
- new net DIP2: R511.1, SW501.2, U504.11 (4B)
- new net IORD: U503.3, U504.1 (1OE), U504.10 (3OE), U504.13 (4OE), U504.4 (2OE)
- new net IOWR: U503.7, U505.11 (LE)
- new net LED0: R507.2, U505.16 (Q3)
- new net LED1: R508.2, U505.17 (Q2)
- new net LED2: R509.2, U505.18 (Q1)
- new net NAUDIO_DATA: J502.4 (Pin_4)
- new net SD_WP: U504.6 (2B)
- new net ~{IOCS}: R514.2, U503.2, U503.6
- new net ~{SD_CD}: U504.3 (1B)
- no-connect marks 0 -> 5
Other:
- note added: "1x Green and 2x Orange side-view reflector LEDs in PLCC2 4x4mm package"
- note added: "Connectors to the Motherboard"
- note added: "Ground pins for measurements"
- note added: "I/O: LEDs & DIP Switches"
- note added: "Mount R514 only if AURA is mounted not (bypass ACS directly to IOCS)."
- note added: "TSSOP-14 4.4x5mm"
- note added: "TSSOP-20 4.4x6.5mm"
- note added: "TSSOP8"
- note added: "dnp"
- note added: "package SOT-23-6"
- note removed: "B-2-B CONNECTOR TO THE MULTIMEDIA BOARD "VA-BO""
- note removed: "TBD: FCDONE not connected"
- company: (none) -> FOR X65.EU DESIGNED BY JSYKORA.INFO
- title: (none) -> OpenX65 - Video/Audio & Ethernet Board
- moved on the sheet: J501, J502, R501, R502, R503, R504, R505, R506, U501
