File: pcb/vabo-rev01/vabo-sheet-06.kicad_sch (KiCad schematic)
At the start: 34 parts, among them SW601 A6SN-4101, U601 ICE5LP1K-SG48, U602 74CBTLV3126PW,118, U603 W25Q16JVSNIQ

Commit message: V/A board rev01 finished and submitted to pcbway
Parts:
- removed C605: 1u, Capacitor_SMD:C_0603_1608Metric_Pad1.08x0.95mm_HandSolder, symbol Device:C_Small
- removed D602, D603, D604: LED, symbol Device:LED
- removed R612, R613, R614: 470, Resistor_SMD:R_0603_1608Metric_Pad0.98x0.95mm_HandSolder, symbol Device:R
- removed R615, R616, R617: 10k, Resistor_SMD:R_0603_1608Metric_Pad0.98x0.95mm_HandSolder, symbol Device:R
- removed SW601: A6SN-4101, Button_Switch_SMD:SW_DIP_SPSTx04_Slide_Omron_A6S-410x_W8.9mm_P2.54mm, symbol Switch:SW_DIP_x04
- added D605: LED_GREEN_0603, LED_SMD:LED_0603_1608Metric_Pad1.05x0.95mm_HandSolder, symbol Device:LED
- added Q601: BSS138, Package_TO_SOT_SMD:SOT-23, symbol Transistor_FET:BSS123
- added R619: 470R, Resistor_SMD:R_0603_1608Metric_Pad0.98x0.95mm_HandSolder, symbol Device:R
- JP601: now left out of the parts list
- U601: value ICE5LP1K-SG48 -> ICE5LP{1,2,4}K-SG48
Connections:
- net DIP is gone; now on net D1: U601.43 (IOT_49a)
- net LED0 is gone; now on net A1: U601.39 (RGB0)
- net LED1 is gone; now on net A0: U601.40 (RGB1)
- net +3V3: now also D605.2 (A)
- net A0: no longer U601.28 (IOT_41a)
- net A1: no longer U601.31 (IOT_42b)
- net A2: now also U601.37 (IOT_45a_G1); no longer U601.32 (IOT_43a)
- net A3: now also U601.38 (IOT_50b); no longer U601.34 (IOT_44b)
- net A4: now also U601.34 (IOT_44b); no longer U601.36 (IOT_48b)
- net A5: no longer U601.37 (IOT_45a_G1)
- net A6: no longer U601.38 (IOT_50b)
- net A7: no longer U601.42 (IOT_51a)
- net AFPGA_CDONE: now also Q601.1 (G)
- net AUDIO_BCK: now also U601.12 (IOB_22b); no longer U601.48 (IOB_4a)
- net AUDIO_DATA: now also U601.13 (IOB_24a); no longer U601.45 (IOB_5b)
- net AUDIO_LRCK: now also U601.18 (IOB_31b); no longer U601.2 (IOB_6a)
- net D0: now also U601.32 (IOT_43a); no longer U601.27 (IOT_38b)
- net D1: no longer U601.26 (IOT_39a)
- net D2: now also U601.44 (IOB_3b_G6); no longer U601.25 (IOT_36b)
- net D3: now also U601.45 (IOB_5b); no longer U601.23 (IOT_37a)
- net D4: now also U601.46 (IOB_0a); no longer U601.21 (IOB_23b)
- net D5: now also U601.47 (IOB_2a); no longer U601.20 (IOB_25b_G3)
- net D6: now also U601.48 (IOB_4a); no longer U601.19 (IOB_29b)
- net D7: now also U601.2 (IOB_6a); no longer U601.18 (IOB_31b)
- net GND: now also Q601.2 (S)
- net VAUDIO_BCK: now also U601.11 (IOB_20a); no longer U601.46 (IOB_0a)
- net VAUDIO_DATA: now also U601.10 (IOB_18a); no longer U601.47 (IOB_2a)
- net VAUDIO_LRCK: now also U601.9 (IOB_16a); no longer U601.44 (IOB_3b_G6)
- net ~{ACS1}: now also U601.26 (IOT_39a); no longer U601.12 (IOB_22b)
- net ~{AIRQ}: now also U601.25 (IOT_36b); no longer U601.6 (IOB_13b)
- net ~{MRD}: now also U601.36 (IOT_48b); no longer U601.9 (IOB_16a)
- net ~{MWR}: now also U601.42 (IOT_51a); no longer U601.10 (IOB_18a)
- net ~{VCS0}: now also U601.28 (IOT_41a); no longer U601.11 (IOB_20a)
- net AFRESB: now reaches R604.2, R607.2, U601.8 (~{CRESET})
- net LED2: no longer names the net of U601.41 (RGB2)
- net SD_WP: no longer names the net of U601.4 (IOB_8a)
- net ~{SD_CD}: no longer names the net of U601.3 (IOB_9b)
- new net: Q601.3 (D), R619.2
- new net: D605.1 (K), R619.1
- new net ~{IOCS}: U601.27 (IOT_38b)
- no-connect marks 0 -> 12
Other:
- note added: ""AURA READY" internal LED"
- note added: "AURA Bypass"
- note added: "For X16 compatiblity, AURA will implement the YM2151 FM-Synthesis (the chip is long out of production). One possible design is JT51 at https://github.com/jotego/jt51 which requires about 2K gates (i.e. ICE5LP2K-SG48 - to be validated)"
- note added: "NOTE: The RGBx pins are open-drain!"
- note added: "R608, R609, R610 mounted only if U601 (AURA) is not."
- note added: "package QFN-48"
- note added: "package SOIC-8 3.9x4.9mm 150mil"
- note added: "package TSSOP-14 4.4x5mm"
- note removed: "R608, R609, R610 mounted only if U601 is not."
- note removed: "TBD: * add CDONE LED * add user btn"
- note removed: "TBD: LED footprint"
- company: (none) -> FOR X65.EU DESIGNED BY JSYKORA.INFO
- title: (none) -> OpenX65 - Video/Audio & Ethernet Board
- moved on the sheet: C601, C602, C603, C604, C606, C607, C608, D601, JP601, R601, R602, R603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
