File: pcb/vabo-rev01/vabo-sheet-07.kicad_sch (KiCad schematic)
At the start: 29 parts, among them J701 Lumberg 1503-07, J702 PINS 1x2, J703 PINS 1x2, Q701 BSS123, SW701 5MS3S102AM6QE, U701 WM8524CGEDT, U702 LM4890MX

Commit message: V/A board rev01 finished and submitted to pcbway
Parts:
- added C712: 3u3, Capacitor_SMD:C_0603_1608Metric_Pad1.08x0.95mm_HandSolder, symbol Device:C_Small
- added C713: 1u, Capacitor_SMD:C_0603_1608Metric_Pad1.08x0.95mm_HandSolder, symbol Device:C_Small
- added C714: 1uF, Capacitor_SMD:C_0603_1608Metric_Pad1.08x0.95mm_HandSolder, symbol Device:C_Small
- added C715, C716: 2n7, Capacitor_SMD:C_0603_1608Metric_Pad1.08x0.95mm_HandSolder, symbol Device:C_Small
- added C717, C718: 4u7, Capacitor_SMD:C_0603_1608Metric_Pad1.08x0.95mm_HandSolder, symbol Device:C_Small
- added C719: 22u/16V, Capacitor_SMD:C_0805_2012Metric_Pad1.18x1.45mm_HandSolder, symbol Device:C
- added R712, R713: 560R, Resistor_SMD:R_0603_1608Metric_Pad0.98x0.95mm_HandSolder, symbol Device:R_Small
- added U703: WM8524CGEDT, Package_SO:TSSOP-16_4.4x5mm_P0.65mm, symbol vera-module:WM8524CGEDT
- C701: value 2.2uF -> 3u3
- C703, C709, C711: value 1uF -> 1u
- C704, C705: value 2.7nF -> 2n7
- C706, C707: value 4.7uF -> 4u7
- Q701: value BSS123 -> BSS138
- R701, R702, R709, R710: value 560 -> 560R
Connections:
- net +3V3: now also C717.1, C718.1, U703.11 (~{MUTE}), U703.12 (AIFMODE), U703.15 (AVDD), U703.6 (LINEVDD)
- net +5V: now also C719.2
- net ASYSCLK: now also U703.10 (MCLK)
- net GND: now also C712.2, C714.2, C715.2, C716.2, C717.2, C718.2, C719.1, U703.13 (AGND), U703.4 (LINEGND)
- net L_AUDIO: now also C715.1, R712.1
- net R_AUDIO: now also C716.1, R713.1
- net LJACK: now reaches J701.T, R710.1
- net SPK1: now reaches C710.2, J702.1 (Pin_1), J703.1 (Pin_1), R704.2, U702.5 (Vo1)
- net SPK2: now reaches J702.2 (Pin_2), J703.2 (Pin_2), U702.8 (Vo2)
- net LINEOUTR: now reaches R702.2, U701.16 (LINEVOUTR)
- net AMPINN: now reaches C708.2, C710.1, R704.1, U702.4 (-IN)
- net RJACK: now reaches J701.R, R709.1
- net LINEOUTL: now reaches R701.2, U701.1 (LINEVOUTL)
- new net: C712.1, U703.14 (VMID)
- new net: C713.1, U703.3 (CPCB)
- new net: C713.2, U703.5 (CPCA)
- new net: C714.1, U703.2 (CPVOUTN)
- new net NAUDIO_BCK: U703.9 (BCLK)
- new net NAUDIO_DATA: U703.7 (DACDAT)
- new net NAUDIO_LRCK: U703.8 (LRCLK)
- new net NLINEOUTL: R712.2, U703.1 (LINEVOUTL)
- new net NLINEOUTR: R713.2, U703.16 (LINEVOUTR)
Other:
- note added: "Audio DAC (PCM/PSG in VERA, FM in AURA)"
- note added: "Audio DAC (Sound from NORA) - optional."
- note added: "dnp"
- note added: "package SOIC-8 3.9x4.9mm"
- note added: "package TSSOP-16 4.4x5mm"
- note removed: "Audio DAC"
- company: (none) -> FOR X65.EU DESIGNED BY JSYKORA.INFO
- title: (none) -> OpenX65 - Video/Audio & Ethernet Board
- moved on the sheet: C708, C709, C710, C711, J701, J702, J703, LS701, Q701, R703, R704, R705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
