File: pcb/vabo-rev01/vabo-sheet-08.kicad_sch (KiCad schematic)
At the start: 43 parts, among them J801 RJ45_Amphenol_RJMG1BD3B8K1ANR, U801 W6100L, Y801 ABM3-25.000MHZ-D2Y-T

Commit message: V/A board rev01 finished and submitted to pcbway
Parts:
- removed R805: 10k, Resistor_SMD:R_0603_1608Metric_Pad0.98x0.95mm_HandSolder, symbol Device:R
- added C816, C817: 22u/16V, Capacitor_SMD:C_0805_2012Metric_Pad1.18x1.45mm_HandSolder, symbol Device:C
- added C818: 1nF/2kV, Capacitor_SMD:C_1206_3216Metric_Pad1.33x1.80mm_HandSolder, symbol Device:C
- J801: value RJ45_Amphenol_RJMG1BD3B8K1ANR -> RJMG1BD3B8K1ANR
- R804: value 10k -> 10M; footprint Resistor_SMD:R_0603_1608Metric_Pad0.98x0.95mm_HandSolder -> Resistor_SMD:R_2512_6332Metric_Pad1.40x3.35mm_HandSolder
Connections:
- net +3V3: now also C816.2, C817.2
- net GND: now also U801.26 (MOD1), U801.28 (MOD3), C816.1, C817.1, C818.2
- net XSCI: now reaches C814.1, R817.2, R820.2, R821.1, U801.12 (XSCI), Y801.2
- net ~{ALED}: now reaches R808.1, U801.20 (~{ACT_LED})
- net LEDYK: now reaches J801.L2 (LEDY_K), R808.2
- net 3V3D: now reaches C808.1, C809.1, FB804.1, R806.1, U801.24 (3V3D), U801.36 (3V3D)
- net ~{WIZRST}: now reaches C815.2, R818.2, R819.2, U801.48 (~{RST})
- net ~{LLED}: now reaches R807.1, U801.17 (~{LNK_LED})
- net LEDGK: now reaches J801.L3 (LEDG_K), R807.2
- net XSCO: now reaches C813.1, R817.1, U801.11 (XSCO), Y801.1
- net CTVDD: now reaches C810.2, FB803.1, J801.L1 (LEDY_A), J801.L4 (LEDG_A), J801.R4 (TCT), J801.R5 (RCT)
- net MOD2: now reaches R806.2, U801.27 (MOD2)
- net MOD0: now reaches R803.1, U801.25 (MOD0)
- net RSET: now reaches R801.1, U801.9 (RSET_BG)
- net LANSH: now reaches J801.13 (SHIELD)
- net LANSH: now also R804.1, C818.1
- no-connect marks 0 -> 4
Other:
- note added: "package LQFP-48"
- company: (none) -> FOR X65.EU DESIGNED BY JSYKORA.INFO
- title: (none) -> OpenX65 - Video/Audio & Ethernet Board
