File: pcb/x65-sbc-revA1/04-rtc_snes.kicad_sch (KiCad schematic)
At the start: 33 parts, among them J403 SNES_Controller_Conn, J404 SNES_Controller_Conn, U401 74LVC2G17DBVR, U402 MCP7940N-xSN, U403 74LVC2G17DBVR, Y402 CM8V-T1A-32.768kHz-9pF-20PPM-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

Commit message: pcb sbc: more pcb work
Parts:
- added D406, D407: LED_GREEN_0603, LED_SMD:LED_0603_1608Metric_Pad1.05x0.95mm_HandSolder, symbol Device:LED
- added R417, R418: 2k7, Resistor_SMD:R_0603_1608Metric_Pad0.98x0.95mm_HandSolder, symbol Device:R
- added R419, R420: 470R, Resistor_SMD:R_0603_1608Metric_Pad0.98x0.95mm_HandSolder, symbol Device:R
- added R421, R422: 33k, Resistor_SMD:R_0603_1608Metric_Pad0.98x0.95mm_HandSolder, symbol Device:R
- added SW401: SW_DIP_x02 TE 1825058-1, Button_Switch_SMD:SW_DIP_SPSTx02_Slide_6.7x6.64mm_W8.61mm_P2.54mm_LowProfile, symbol Switch:SW_DIP_x02
Connections:
- net +3V3: now also D406.2 (A), D407.2 (A), R421.2, R422.2
- new net: D407.1 (K), R420.2
- new net: R417.1, SW401.4
- new net: SW401.1, SW401.2
- new net: R418.1, SW401.3
- new net: D406.1 (K), R419.2
- new net DIPLED0: R417.2, R419.1, R421.1
- new net DIPLED1: R418.2, R420.1, R422.1
Other:
- note added: "RTC/MCP7940N I2C DEVICE ADDRESS (8b=shifted) = 0b1101_111W = 0xDE, that is 7-bit addr 0x6F PS2 CONTROLLER (IN NORA) I2C DEVICE ADDRESS (8b=shifted) = 0b1000010W = 0x84, that is 7-bit addr 0x42"
- note removed: "RTC/MCP7940N I2C DEVICE ADDRESS (8b=shifted) = 0b1101_111W = 0xDE PS2 CONTROLLER (IN NORA) I2C DECICE ADDRESS (8b=shifted) = 0b1000010W = 0x84"
- moved on the sheet: D402, D403, R401, R402, R413, R414, R415, R416

Commit message: x65-sbc: pcb done
Parts:
- removed C405: 1u, Capacitor_SMD:C_0603_1608Metric_Pad1.08x0.95mm_HandSolder, symbol Device:C
Connections:
- net GND: now also SW401.1, SW401.2
Other:
- moved on the sheet: C404
Changed lines of the file:
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@@
   (title_block
     (title "X65-SBC")
-    (date "2023-12-29")
+    (date "2024-01-10")
     (rev "revA1")
     (company "FOR X65.EU DESIGNED BY JSYKORA.INFO")
@@
   (junction (at 238.76 69.85) (diameter 0) (color 0 0 0 0)
   )
-  (junction (at 227.33 110.49) (diameter 0) (color 0 0 0 0)
-  )
   (junction (at 215.265 79.375) (diameter 0) (color 0 0 0 0)
   )
@@
   (junction (at 108.585 84.455) (diameter 0) (color 0 0 0 0)
   )
+  (junction (at 146.05 38.1) (diameter 0) (color 0 0 0 0)
+  )
   (junction (at 90.17 53.34) (diameter 0) (color 0 0 0 0)
   )
@@
     (stroke (width 0) (type default))
   )
+  (wire (pts (xy 136.525 38.1) (xy 146.05 38.1))
+    (stroke (width 0) (type default))
+  )
   (wire (pts (xy 43.815 142.875) (xy 43.815 146.685))
     (stroke (width 0) (type default))
@@
     (stroke (width 0) (type default))
   )
-  (wire (pts (xy 224.155 110.49) (xy 227.33 110.49))
+  (wire (pts (xy 59.055 35.56) (xy 62.865 35.56))
     (stroke (width 0) (type default))
   )
-  (wire (pts (xy 59.055 35.56) (xy 62.865 35.56))
+  (wire (pts (xy 136.525 42.545) (xy 136.525 38.1))
     (stroke (width 0) (type default))
   )
@@
     (stroke (width 0) (type default))
   )
-  (wire (pts (xy 227.33 110.49) (xy 231.14 110.49))
+  (wire (pts (xy 224.155 110.49) (xy 231.14 110.49))
     (stroke (width 0) (type default))
   )
@@
     (stroke (width 0) (type default))
   )
-  (wire (pts (xy 33.02 92.075) (xy 33.02 94.615))
+  (wire (pts (xy 33.02 92.075) (xy 33.02 95.25))
     (stroke (width 0) (type default))
   )
@@
     )
   )
-  (symbol (lib_id "Device:C") (at 227.33 114.3 0) (unit 1)
-    (in_bom yes) (on_board yes) (dnp no)
-    (property "Reference" "C405" (at 219.71 115.57 0)
-      (effects (font (size 1.27 1.27)) (justify left))
-    )
-    (property "Value" "1u" (at 219.71 118.11 0)
-      (effects (font (size 1.27 1.27)) (justify left))
-    )
-    (property "Footprint" "Capacitor_SMD:C_0603_1608Metric_Pad1.08x0.95mm_HandSolder" (at 228.2952 118.11 0)
-      (effects (font (size 1.27 1.27)) hide)
-    )
-    (property "Datasheet" "~" (at 227.33 114.3 0)
-      (effects (font (size 1.27 1.27)) hide)
-    )
-    (pin "1")
-    (pin "2")
-    (instances
-      (project "x65-sbc-revA1"
-        (path "/85750bea-43a1-4629-9575-611e72af7f9f/a0a926f8-222f-4537-8c1a-4e84db3f94e8"
-          (reference "C405") (unit 1)
-        )
-      )
-    )
-  )
   (symbol (lib_id "power:+5V") (at 146.05 38.1 0) (unit 1)
     (in_bom yes) (on_board yes) (dnp no)
@@
     )
   )
-  (symbol (lib_name "GND_1") (lib_id "power:GND") (at 227.33 118.11 0) (unit 1)
-    (in_bom yes) (on_board yes) (dnp no) (fields_autoplaced)
-    (property "Reference" "#PWR0422" (at 227.33 124.46 0)
-      (effects (font (size 1.27 1.27)) hide)
-    )
-    (property "Value" "GND" (at 227.33 122.555 0)
-      (effects (font (size 1.27 1.27)))
-    )
-    (property "Footprint" "" (at 227.33 118.11 0)
-      (effects (font (size 1.27 1.27)) hide)
-    )
-    (property "Datasheet" "" (at 227.33 118.11 0)
-      (effects (font (size 1.27 1.27)) hide)
-    )
-    (pin "1")
-    (instances
-      (project "x65-sbc-revA1"
-        (path "/85750bea-43a1-4629-9575-611e72af7f9f/a0a926f8-222f-4537-8c1a-4e84db3f94e8"
-          (reference "#PWR0422") (unit 1)
-        )
-      )
-    )
-  )
   (symbol (lib_id "Device:R") (at 43.815 139.065 180) (unit 1)
     (in_bom yes) (on_board yes) (dnp no)
@@
     )
   )
-  (symbol (lib_id "Device:C") (at 210.82 135.255 0) (unit 1)
+  (symbol (lib_id "Device:C") (at 136.525 46.355 0) (mirror y) (unit 1)
     (in_bom yes) (on_board yes) (dnp no) (fields_autoplaced)
-    (property "Reference" "C404" (at 214.63 133.9849 0)
+    (property "Reference" "C404" (at 132.715 45.0849 0)
       (effects (font (size 1.27 1.27)) (justify left))
     )
-    (property "Value" "1u" (at 214.63 136.5249 0)
+    (property "Value" "1u" (at 132.715 47.6249 0)
       (effects (font (size 1.27 1.27)) (justify left))
     )
-    (property "Footprint" "Capacitor_SMD:C_0603_1608Metric_Pad1.08x0.95mm_HandSolder" (at 211.7852 139.065 0)
+    (property "Footprint" "Capacitor_SMD:C_0603_1608Metric_Pad1.08x0.95mm_HandSolder" (at 135.5598 50.165 0)
       (effects (font (size 1.27 1.27)) hide)
     )
-    (property "Datasheet" "~" (at 210.82 135.255 0)
+    (property "Datasheet" "~" (at 136.525 46.355 0)
       (effects (font (size 1.27 1.27)) hide)
     )
@@
     )
   )
-  (symbol (lib_name "GND_1") (lib_id "power:GND") (at 210.82 139.065 0) (unit 1)
+  (symbol (lib_name "GND_1") (lib_id "power:GND") (at 136.525 50.165 0) (mirror y) (unit 1)
     (in_bom yes) (on_board yes) (dnp no) (fields_autoplaced)
-    (property "Reference" "#PWR0421" (at 210.82 145.415 0)
+    (property "Reference" "#PWR0421" (at 136.525 56.515 0)
       (effects (font (size 1.27 1.27)) hide)
     )
-    (property "Value" "GND" (at 210.82 143.51 0)
+    (property "Value" "GND" (at 136.525 54.61 0)
       (effects (font (size 1.27 1.27)))
     )
-    (property "Footprint" "" (at 210.82 139.065 0)
+    (property "Footprint" "" (at 136.525 50.165 0)
       (effects (font (size 1.27 1.27)) hide)
     )
-    (property "Datasheet" "" (at 210.82 139.065 0)
+    (property "Datasheet" "" (at 136.525 50.165 0)
       (effects (font (size 1.27 1.27)) hide)
     )
@@
         )
       )
-    )
-  )
-  (symbol (lib_id "power:+5V") (at 210.82 131.445 0) (unit 1)
-    (in_bom yes) (on_board yes) (dnp no)
-    (property "Reference" "#PWR0420" (at 210.82 135.255 0)
-      (effects (font (size 1.27 1.27)) hide)
-    )
-    (property "Value" "+5V" (at 210.82 127.635 0)
-      (effects (font (size 1.27 1.27)))
-    )
-    (property "Footprint" "" (at 210.82 131.445 0)
-      (effects (font (size 1.27 1.27)) hide)
-    )
-    (property "Datasheet" "" (at 210.82 131.445 0)
-      (effects (font (size 1.27 1.27)) hide)
-    )
-    (pin "1")
-    (instances
-      (project "x65-sbc-revA1"
-        (path "/85750bea-43a1-4629-9575-611e72af7f9f/a0a926f8-222f-4537-8c1a-4e84db3f94e8"
-          (reference "#PWR0420") (unit 1)
-        )
-      )
