File: pcb/x65-sbc-revA1/06-ps2_uext.kicad_sch (KiCad schematic)
At the start: 29 parts, among them J601 PINS 2x10p 2,54mm, J603 DS1013-10RSIB CONNFLY, J605 TE 5749180-1, J606 TE 5749180-1, Q601 BSS138, Q602 BSS138, Q603 BSS138, Q604 BSS138

Commit message: pcb sbc: more pcb work
Parts:
- added D301: CUS10S30,H3F, Diode_SMD:D_SOD-323_HandSoldering, symbol Device:D_Schottky
- added JP701: SolderJumper_2_Bridged, Jumper:SolderJumper-2_P1.3mm_Open_RoundedPad1.0x1.5mm, symbol Jumper:SolderJumper_2_Open
- J601: value PINS 2x10p 2,54mm -> IDC PINS 2x10p 2,54mm; footprint Connector_PinHeader_2.54mm:PinHeader_2x10_P2.54mm_Vertical -> Connector_IDC:IDC-Header_2x10_P2.54mm_Vertical
- R618, R619: value 0R -> 100R
Connections:
- net +3V3: now also D301.2 (A)
- net +5V: now also JP701.2 (B)
- net A5 renamed UEPWR
- net UEPWR: now also D301.1 (K), JP701.1 (A)

Commit message: x65-sbc: pcb done
Parts:
- JP601: renamed from JP701; value SolderJumper_2_Bridged -> SolderJumper_2_Open
- renumbered D301 to D603, D301 to D604
Changed lines of the file:
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@@
   (title_block
     (title "X65-SBC")
-    (date "2023-12-29")
+    (date "2024-01-10")
     (rev "revA1")
     (company "FOR X65.EU DESIGNED BY JSYKORA.INFO")
@@
   (symbol (lib_id "Device:D_Schottky") (at 47.625 61.595 180) (unit 1)
     (in_bom yes) (on_board yes) (dnp no) (fields_autoplaced)
-    (property "Reference" "D301" (at 47.9425 55.88 0)
+    (property "Reference" "D604" (at 47.9425 55.88 0)
       (effects (font (size 1.27 1.27)))
     )
@@
     (instances
       (project "x65-sbc-revA1"
-        (path "/85750bea-43a1-4629-9575-611e72af7f9f/17c238d7-f888-4cc2-8790-8144029e69c2"
-          (reference "D301") (unit 1)
-        )
         (path "/85750bea-43a1-4629-9575-611e72af7f9f/9450b3cd-ef01-4353-a64a-2812b3ee45c9"
           (reference "D604") (unit 1)
@@
   (symbol (lib_id "power:+5V") (at 40.64 69.215 0) (unit 1)
     (in_bom yes) (on_board yes) (dnp no)
-    (property "Reference" "#PWR0712" (at 40.64 73.025 0)
+    (property "Reference" "#PWR0607" (at 40.64 73.025 0)
       (effects (font (size 1.27 1.27)) hide)
     )
@@
     (instances
       (project "x65-sbc-revA1"
-        (path "/85750bea-43a1-4629-9575-611e72af7f9f/a59c40b6-4c79-43f8-90db-e6d1d1476407"
-          (reference "#PWR0712") (unit 1)
-        )
         (path "/85750bea-43a1-4629-9575-611e72af7f9f/9450b3cd-ef01-4353-a64a-2812b3ee45c9"
           (reference "#PWR0607") (unit 1)
@@
   (symbol (lib_id "Jumper:SolderJumper_2_Open") (at 47.625 69.85 180) (unit 1)
     (in_bom no) (on_board yes) (dnp no)
-    (property "Reference" "JP701" (at 47.625 67.31 0)
+    (property "Reference" "JP601" (at 47.625 67.31 0)
       (effects (font (size 1.27 1.27)))
     )
-    (property "Value" "SolderJumper_2_Bridged" (at 53.34 66.675 0)
+    (property "Value" "SolderJumper_2_Open" (at 53.34 66.675 0)
       (effects (font (size 1 1)) hide)
     )
@@
     (instances
       (project "x65-sbc-revA1"
-        (path "/85750bea-43a1-4629-9575-611e72af7f9f/a59c40b6-4c79-43f8-90db-e6d1d1476407"
-          (reference "JP701") (unit 1)
-        )
         (path "/85750bea-43a1-4629-9575-611e72af7f9f/9450b3cd-ef01-4353-a64a-2812b3ee45c9"
           (reference "JP601") (unit 1)
@@
   (symbol (lib_id "Device:C") (at 183.515 121.92 0) (unit 1)
     (in_bom yes) (on_board yes) (dnp no)
-    (property "Reference" "C602" (at 177.8 120.65 0)
+    (property "Reference" "C602" (at 177.8 119.38 0)
       (effects (font (size 1.27 1.27)) (justify left))
     )
-    (property "Value" "1u" (at 177.8 123.19 0)
+    (property "Value" "1u" (at 177.8 121.92 0)
       (effects (font (size 1.27 1.27)) (justify left))
     )
@@
   (symbol (lib_id "Device:C") (at 174.625 27.305 0) (unit 1)
     (in_bom yes) (on_board yes) (dnp no)
-    (property "Reference" "C601" (at 168.91 26.035 0)
+    (property "Reference" "C601" (at 168.91 24.765 0)
       (effects (font (size 1.27 1.27)) (justify left))
     )
-    (property "Value" "1u" (at 168.91 28.575 0)
+    (property "Value" "1u" (at 168.91 27.305 0)
       (effects (font (size 1.27 1.27)) (justify left))
     )
@@
   (symbol (lib_id "Device:D_Schottky") (at 96.52 121.92 90) (unit 1)
     (in_bom yes) (on_board yes) (dnp no) (fields_autoplaced)
-    (property "Reference" "D301" (at 99.06 120.9674 90)
+    (property "Reference" "D603" (at 99.06 120.9674 90)
       (effects (font (size 1.27 1.27)) (justify right))
     )
@@
     (instances
       (project "x65-sbc-revA1"
-        (path "/85750bea-43a1-4629-9575-611e72af7f9f/17c238d7-f888-4cc2-8790-8144029e69c2"
-          (reference "D301") (unit 1)
-        )
         (path "/85750bea-43a1-4629-9575-611e72af7f9f/9450b3cd-ef01-4353-a64a-2812b3ee45c9"
           (reference "D603") (unit 1)
