File: pcb/x65-sbc-revA1/07-pwrsup.kicad_sch (KiCad schematic)
At the start: 22 parts, among them J701 Conn_01x02, J702 Conn_01x01, J703 Conn_01x01, U701 MP2149GJ

Commit message: pcb sbc: more pcb work
Parts:
- D701: value AA4040LCGCK-AMT -> LED_GREEN_0603; footprint ledplcc2:PLCC2_4x4mm -> LED_SMD:LED_0603_1608Metric_Pad1.05x0.95mm_HandSolder
Other:
- note removed: "JP701, 702 = make closed by default??"
Changed lines of the file:
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@@
     (effects (font (size 1.27 1.27)) (justify left bottom))
-  )
-  (text "JP701, 702 = make closed by default??" (at 60.325 160.02 0)
-    (effects (font (size 1.27 1.27) (color 255 0 0 1)) (justify left bottom))
   )
   (text "Alternative power input connector" (at 63.5 125.73 0)
@@
       (effects (font (size 1.27 1.27)) (justify right))
     )
-    (property "Value" "AA4040LCGCK-AMT" (at 60.96 80.3274 90)
+    (property "Value" "LED_GREEN_0603" (at 60.96 80.3274 90)
       (effects (font (size 1.27 1.27)) (justify right))
     )
-    (property "Footprint" "ledplcc2:PLCC2_4x4mm" (at 57.15 77.47 0)
-      (effects (font (size 1.27 1.27)) hide)
-    )
+    (property "Footprint" "LED_SMD:LED_0603_1608Metric_Pad1.05x0.95mm_HandSolder" (at 57.15 77.47 0)
+      (effects (font (size 1.27 1.27)) hide)
+    )

Commit message: x65-sbc: pcb done
Parts:
- added J704: Conn_01x01, Connector_PinHeader_2.54mm:PinHeader_1x01_P2.54mm_Vertical, symbol Connector_Generic:Conn_01x01
- renumbered C510 to C705
Connections:
- net GND: now also J704.1 (Pin_1)
Changed lines of the file:
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@@
   (title_block
     (title "X65-SBC")
-    (date "2023-12-29")
+    (date "2024-01-10")
     (rev "revA1")
     (company "FOR X65.EU DESIGNED BY JSYKORA.INFO")
@@
   (symbol (lib_id "Device:C") (at 97.155 47.625 0) (unit 1)
     (in_bom yes) (on_board yes) (dnp no)
-    (property "Reference" "C510" (at 89.535 46.355 0)
+    (property "Reference" "C705" (at 89.535 46.355 0)
       (effects (font (size 1.27 1.27)) (justify left))
     )
@@
     (instances
       (project "x65-sbc-revA1"
-        (path "/85750bea-43a1-4629-9575-611e72af7f9f/3a4f5a92-8b22-4d71-ac4e-37e2fe30ebbe"
-          (reference "C510") (unit 1)
-        )
         (path "/85750bea-43a1-4629-9575-611e72af7f9f/a59c40b6-4c79-43f8-90db-e6d1d1476407"
           (reference "C705") (unit 1)
@@
     )
   )
+  (symbol (lib_id "power:GND") (at 114.3 147.32 270) (unit 1)
+    (in_bom yes) (on_board yes) (dnp no)
+    (property "Reference" "#PWR0718" (at 107.95 147.32 0)
+      (effects (font (size 1.27 1.27)) hide)
+    )
+    (property "Value" "GND" (at 106.68 147.32 90)
+      (effects (font (size 1.27 1.27)) (justify left))
+    )
+    (property "Footprint" "" (at 114.3 147.32 0)
+      (effects (font (size 1.27 1.27)) hide)
+    )
+    (property "Datasheet" "" (at 114.3 147.32 0)
+      (effects (font (size 1.27 1.27)) hide)
+    )
+    (pin "1")
+    (instances
+      (project "x65-sbc-revA1"
+        (path "/85750bea-43a1-4629-9575-611e72af7f9f/a59c40b6-4c79-43f8-90db-e6d1d1476407"
+          (reference "#PWR0718") (unit 1)
+        )
+      )
+    )
+  )
   (symbol (lib_id "Device:C") (at 137.795 54.61 90) (unit 1)
     (in_bom yes) (on_board yes) (dnp no)
@@
         )
       )
+    )
+  )
+  (symbol (lib_id "Connector_Generic:Conn_01x01") (at 119.38 147.32 0) (unit 1)
+    (in_bom no) (on_board yes) (dnp yes) (fields_autoplaced)
+    (property "Reference" "J704" (at 121.92 146.0499 0)
+      (effects (font (size 1.27 1.27)) (justify left))
+    )
+    (property "Value" "Conn_01x01" (at 121.92 148.5899 0)
+      (effects (font (size 1.27 1.27)) (justify left))
+    )
+    (property "Footprint" "Connector_PinHeader_2.54mm:PinHeader_1x01_P2.54mm_Vertical" (at 119.38 147.32 0)
+      (effects (font (size 1.27 1.27)) hide)
+    )
+    (property "Datasheet" "~" (at 119.38 147.32 0)
+      (effects (font (size 1.27 1.27)) hide)
+    )
+    (pin "1")
+    (instances
+      (project "x65-sbc-revA1"
+        (path "/85750bea-43a1-4629-9575-611e72af7f9f/a59c40b6-4c79-43f8-90db-e6d1d1476407"
+          (reference "J704") (unit 1)
+        )
+      )
