File: pcb/x65-sbc-revA1/08-vera_fpga.kicad_sch (KiCad schematic)
At the start: 43 parts, among them J303 ICD15S13E4GV00LF, Q801 BSS138, U801 ICE40UP5K-SG48ITR50, X801 SG5032CAN_25.000000M-TJGA3

Commit message: pcb sbc: more pcb work
Parts:
- removed R801, R807: 0R, Resistor_SMD:R_0603_1608Metric_Pad0.98x0.95mm_HandSolder, symbol Device:R
Connections:
- net VFPGA_CRESB is gone; now on net ~{VRST}: R802.2, U801.8 (CRESET_B)
- net 25MHZ renamed 25MHz
Changed lines of the file:
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@@
     (stroke (width 0) (type default))
   )
-  (wire (pts (xy 236.22 36.83) (xy 239.395 36.83))
-    (stroke (width 0) (type default))
-  )
   (wire (pts (xy 234.95 99.695) (xy 231.14 99.695))
     (stroke (width 0) (type default))
@@
     (stroke (width 0) (type default))
   )
-  (wire (pts (xy 29.845 76.835) (xy 32.385 76.835))
-    (stroke (width 0) (type default))
-  )
   (wire (pts (xy 141.605 107.315) (xy 149.225 107.315))
     (stroke (width 0) (type default))
@@
     (stroke (width 0) (type default))
   )
-  (wire (pts (xy 247.015 36.83) (xy 252.73 36.83))
+  (wire (pts (xy 236.22 36.83) (xy 252.73 36.83))
     (stroke (width 0) (type default))
   )
@@
     (stroke (width 0) (type default))
   )
-  (wire (pts (xy 40.005 76.835) (xy 43.815 76.835))
+  (wire (pts (xy 37.465 76.835) (xy 43.815 76.835))
     (stroke (width 0) (type default))
   )
@@
     (effects (font (size 1.27 1.27)) (justify left bottom))
   )
-  (label "VFPGA_CRESB" (at 49.53 76.835 0) (fields_autoplaced)
-    (effects (font (size 1.27 1.27)) (justify left bottom))
-  )
   (label "D4" (at 66.675 109.855 0) (fields_autoplaced)
     (effects (font (size 1.27 1.27)) (justify left bottom))
@@
     (effects (font (size 1.27 1.27)) (justify left bottom))
   )
-  (label "25MHZ" (at 236.22 34.925 90) (fields_autoplaced)
-    (effects (font (size 1.27 1.27)) (justify left bottom))
-  )
   (label "D6" (at 66.675 104.775 0) (fields_autoplaced)
     (effects (font (size 1.27 1.27)) (justify left bottom))
@@
     )
   )
-  (global_label "~{VRST}" (shape input) (at 29.845 76.835 180) (fields_autoplaced)
+  (global_label "~{VRST}" (shape input) (at 37.465 76.835 180) (fields_autoplaced)
     (effects (font (size 1.27 1.27)) (justify right))
-    (property "Intersheetrefs" "${INTERSHEET_REFS}" (at 22.8962 76.7556 0)
+    (property "Intersheetrefs" "${INTERSHEET_REFS}" (at 30.5162 76.7556 0)
       (effects (font (size 1.27 1.27)) (justify right) hide)
     )
@@
     )
   )
-  (global_label "ESYSCLK" (shape output) (at 252.73 36.83 0) (fields_autoplaced)
+  (global_label "25MHz" (shape output) (at 252.73 36.83 0) (fields_autoplaced)
     (effects (font (size 1.27 1.27)) (justify left))
-    (property "Intersheetrefs" "${INTERSHEET_REFS}" (at 263.3679 36.7506 0)
+    (property "Intersheetrefs" "${INTERSHEET_REFS}" (at 261.9442 36.83 0)
       (effects (font (size 1.27 1.27)) (justify left) hide)
     )
@@
     )
   )
-  (symbol (lib_id "Device:R") (at 243.205 36.83 90) (unit 1)
-    (in_bom yes) (on_board yes) (dnp no)
-    (property "Reference" "R807" (at 243.205 34.29 90)
-      (effects (font (size 1.27 1.27)))
-    )
-    (property "Value" "0R" (at 243.205 36.83 90)
-      (effects (font (size 1.27 1.27)))
-    )
-    (property "Footprint" "Resistor_SMD:R_0603_1608Metric_Pad0.98x0.95mm_HandSolder" (at 243.205 38.608 90)
-      (effects (font (size 1.27 1.27)) hide)
-    )
-    (property "Datasheet" "~" (at 243.205 36.83 0)
-      (effects (font (size 1.27 1.27)) hide)
-    )
-    (pin "1")
-    (pin "2")
-    (instances
-      (project "x65-sbc-revA1"
-        (path "/85750bea-43a1-4629-9575-611e72af7f9f/ccadd080-4540-46b4-871b-c090a4eaa310"
-          (reference "R807") (unit 1)
-        )
-      )
-      (project "openX65-vabo"
-        (path "/b8085944-4b3e-4781-a52b-94fe64f9a100/06b8d5f1-9178-4323-97c4-d131b7dff649"
-          (reference "R206") (unit 1)
-        )
-      )
-    )
-  )
   (symbol (lib_id "vera-module:ICE40UP5K-SG48ITR50") (at 90.805 48.895 0) (unit 1)
     (in_bom yes) (on_board yes) (dnp no)
@@
         )
       )
-    )
-  )
-  (symbol (lib_id "Device:R") (at 36.195 76.835 90) (unit 1)
-    (in_bom yes) (on_board yes) (dnp no) (fields_autoplaced)
-    (property "Reference" "R801" (at 36.195 71.12 90)
-      (effects (font (size 1.27 1.27)))
-    )
-    (property "Value" "0R" (at 36.195 73.66 90)
-      (effects (font (size 1.27 1.27)))
-    )
-    (property "Footprint" "Resistor_SMD:R_0603_1608Metric_Pad0.98x0.95mm_HandSolder" (at 36.195 78.613 90)
-      (effects (font (size 1.27 1.27)) hide)
-    )
-    (property "Datasheet" "~" (at 36.195 76.835 0)
-      (effects (font (size 1.27 1.27)) hide)
-    )
-    (pin "1")
-    (pin "2")
-    (instances
-      (project "x65-sbc-revA1"
-        (path "/85750bea-43a1-4629-9575-611e72af7f9f/ccadd080-4540-46b4-871b-c090a4eaa310"
-          (reference "R801") (unit 1)
-        )
-      )
-      (project "openX65-vabo"
-        (path "/b8085944-4b3e-4781-a52b-94fe64f9a100/06b8d5f1-9178-4323-97c4-d131b7dff649"
-          (reference "R208") (unit 1)
-        )
-      )

Commit message: x65-sbc: pcb done
Parts:
- renumbered J303 to J801, R309 to R808, R310 to R809, R311 to R810, R312 to R811, R313 to R812, R314 to R813, R315 to R814, R316 to R815, R317 to R816, R318 to R817, R319 to R818, R320 to R819, R323 to R820, R324 to R821, R325 to R822, R326 to R823, R327 to R824, R328 to R825, R329 to R826, R330 to R827, R331 to R828, R321 to R829, R322 to R830
