File: pcb/x65-sbc-revA1/09-sdcard.kicad_sch (KiCad schematic)
At the start: 22 parts, among them J901 DM1AA-SF-PEJ, U901 74CBTLV3126PW,118, U902 74CBTLV3126PW,118, U903 74AHC00PW, U904 W25Q16JVSNIQ

Commit message: x65-sbc: pcb done
Parts:
- removed C904: 1u, Capacitor_SMD:C_0603_1608Metric_Pad1.08x0.95mm_HandSolder, symbol Device:C_Small
Other:
- note added: "Secure Digital Interface"
- note removed: "Secure Digital Interface - like an "FDD""
Changed lines of the file:
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@@
   (title_block
     (title "X65-SBC")
-    (date "2023-12-29")
+    (date "2024-01-10")
     (rev "revA1")
     (company "FOR X65.EU DESIGNED BY JSYKORA.INFO")
@@
     (stroke (width 0) (type default))
   )
-  (polyline (pts (xy 167.64 71.12) (xy 167.64 76.2))
+  (polyline (pts (xy 167.64 71.755) (xy 167.64 76.835))
     (stroke (width 0) (type default))
   )
@@
     (effects (font (size 1.27 1.27)) (justify left bottom))
   )
-  (text "Secure Digital Interface - like an \"FDD\"" (at 29.21 121.92 0)
+  (text "Secure Digital Interface" (at 39.37 121.92 0)
     (effects (font (size 2 2)) (justify left bottom))
   )
@@
         (path "/b8085944-4b3e-4781-a52b-94fe64f9a100/24ab6e58-c39a-4580-a4ca-24b4eca62ff3"
           (reference "#PWR0410") (unit 1)
-        )
-      )
-    )
-  )
-  (symbol (lib_id "Device:C_Small") (at 226.06 45.72 0) (unit 1)
-    (in_bom yes) (on_board yes) (dnp no)
-    (property "Reference" "C904" (at 228.3968 44.5516 0)
-      (effects (font (size 1.27 1.27)) (justify left))
-    )
-    (property "Value" "1u" (at 228.3968 46.863 0)
-      (effects (font (size 1.27 1.27)) (justify left))
-    )
-    (property "Footprint" "Capacitor_SMD:C_0603_1608Metric_Pad1.08x0.95mm_HandSolder" (at 226.06 45.72 0)
-      (effects (font (size 1.27 1.27)) hide)
-    )
-    (property "Datasheet" "~" (at 226.06 45.72 0)
-      (effects (font (size 1.27 1.27)) hide)
-    )
-    (pin "1")
-    (pin "2")
-    (instances
-      (project "x65-sbc-revA1"
-        (path "/85750bea-43a1-4629-9575-611e72af7f9f/00150742-fc5e-4d8a-b33f-e79b4d66582a"
-          (reference "C904") (unit 1)
-        )
-      )
-      (project "openX65-vabo"
-        (path "/b8085944-4b3e-4781-a52b-94fe64f9a100/24ab6e58-c39a-4580-a4ca-24b4eca62ff3"
-          (reference "C404") (unit 1)
         )
       )
@@
     )
   )
-  (symbol (lib_id "power:+3V3") (at 226.06 43.18 0) (mirror y) (unit 1)
-    (in_bom yes) (on_board yes) (dnp no)
-    (property "Reference" "#PWR0923" (at 226.06 46.99 0)
-      (effects (font (size 1.27 1.27)) hide)
-    )
-    (property "Value" "+3V3" (at 225.679 38.7858 0)
-      (effects (font (size 1.27 1.27)))
-    )
-    (property "Footprint" "" (at 226.06 43.18 0)
-      (effects (font (size 1.27 1.27)) hide)
-    )
-    (property "Datasheet" "" (at 226.06 43.18 0)
-      (effects (font (size 1.27 1.27)) hide)
-    )
-    (pin "1")
-    (instances
-      (project "x65-sbc-revA1"
-        (path "/85750bea-43a1-4629-9575-611e72af7f9f/00150742-fc5e-4d8a-b33f-e79b4d66582a"
-          (reference "#PWR0923") (unit 1)
-        )
-      )
-      (project "openX65-vabo"
-        (path "/b8085944-4b3e-4781-a52b-94fe64f9a100/24ab6e58-c39a-4580-a4ca-24b4eca62ff3"
-          (reference "#PWR0418") (unit 1)
-        )
-      )
-    )
-  )
   (symbol (lib_id "Device:R_Small") (at 253.365 121.285 270) (unit 1)
     (in_bom yes) (on_board yes) (dnp no)
@@
         )
       )
-    )
-  )
-  (symbol (lib_id "power:GND") (at 226.06 48.26 0) (mirror y) (unit 1)
-    (in_bom yes) (on_board yes) (dnp no)
-    (property "Reference" "#PWR0924" (at 226.06 54.61 0)
-      (effects (font (size 1.27 1.27)) hide)
-    )
-    (property "Value" "GND" (at 225.933 52.6542 0)
-      (effects (font (size 1.27 1.27)))
-    )
-    (property "Footprint" "" (at 226.06 48.26 0)
-      (effects (font (size 1.27 1.27)) hide)
-    )
-    (property "Datasheet" "" (at 226.06 48.26 0)
-      (effects (font (size 1.27 1.27)) hide)
-    )
-    (pin "1")
-    (instances
-      (project "x65-sbc-revA1"
-        (path "/85750bea-43a1-4629-9575-611e72af7f9f/00150742-fc5e-4d8a-b33f-e79b4d66582a"
-          (reference "#PWR0924") (unit 1)
-        )
-      )
-      (project "openX65-vabo"
-        (path "/b8085944-4b3e-4781-a52b-94fe64f9a100/24ab6e58-c39a-4580-a4ca-24b4eca62ff3"
-          (reference "#PWR0419") (unit 1)
-        )
-      )
