File: pcb/x65-sbc-revA1/10-aura_fpga.kicad_sch (KiCad schematic)
At the start: 28 parts, among them Q1001 BSS138, U1001 ICE40UP5K-SG48ITR50, U1002 74CBTLV3126PW,118, U1003 W25Q16JVSNIQ

Commit message: pcb sbc: more pcb work
Parts:
- removed R1005: 0R, Resistor_SMD:R_0603_1608Metric_Pad0.98x0.95mm_HandSolder, symbol Device:R
- added R415: 470R, Resistor_SMD:R_0603_1608Metric_Pad0.98x0.95mm_HandSolder, symbol Device:R
Connections:
- net AFRESB is gone; now on net ~{ARST}: R1006.2, U1001.8 (~{CRESET})
- net A0: now also U1001.45 (IOB_5b); no longer U1001.40 (RGB1)
- net A1: now also U1001.18 (IOB_31b); no longer U1001.39 (RGB0)
- net A2: now also U1001.19 (IOB_29b); no longer U1001.37 (IOT_45a_G1)
- net A3: now also U1001.13 (IOB_24a); no longer U1001.38 (IOT_50b)
- net A4: now also U1001.21 (IOB_23b); no longer U1001.34 (IOT_44b)
- net AUDIO_BCK: now also U1001.9 (IOB_16a); no longer U1001.12 (IOB_22b)
- net AUDIO_DATA: now also U1001.3 (IOB_9b); no longer U1001.13 (IOB_24a)
- net AUDIO_LRCK: now also U1001.4 (IOB_8a); no longer U1001.18 (IOB_31b)
- net AURALED: now also U1001.42 (IOT_51a); no longer U1001.31 (IOT_42b)
- net D0: now also U1001.25 (IOT_36b); no longer U1001.32 (IOT_43a)
- net D1: now also U1001.26 (IOT_39a); no longer U1001.43 (IOT_49a)
- net D2: now also U1001.27 (IOT_38b); no longer U1001.44 (IOB_3b_G6)
- net D3: now also U1001.31 (IOT_42b); no longer U1001.45 (IOB_5b)
- net D4: now also U1001.32 (IOT_43a); no longer U1001.46 (IOB_0a)
- net D5: now also U1001.34 (IOT_44b); no longer U1001.47 (IOB_2a)
- net D6: now also U1001.36 (IOT_48b); no longer U1001.48 (IOB_4a)
- net D7: now also U1001.37 (IOT_45a_G1); no longer U1001.2 (IOB_6a)
- net VAUDIO_BCK: now also U1001.12 (IOB_22b); no longer U1001.11 (IOB_20a)
- net VAUDIO_DATA: now also U1001.11 (IOB_20a); no longer U1001.10 (IOB_18a)
- net VAUDIO_LRCK: now also U1001.10 (IOB_18a); no longer U1001.9 (IOB_16a)
- net ~{ACS1}: now also U1001.46 (IOB_0a), R415.1; no longer U1001.26 (IOT_39a)
- net ~{AIRQ}: now also U1001.48 (IOB_4a); no longer U1001.25 (IOT_36b)
- net ~{MRD}: now also U1001.20 (IOB_25b_G3); no longer U1001.36 (IOT_48b)
- net ~{MUTE}: now also U1001.38 (IOT_50b); no longer U1001.3 (IOB_9b)
- net ~{MWR}: now also U1001.23 (IOT_37a); no longer U1001.42 (IOT_51a)
- net ~{SD_SSEL}: now also U1001.43 (IOT_49a); no longer U1001.27 (IOT_38b)
- net at D402.1 (K), R415.2: now also R415.2
- no-connect marks 7 -> 4
Other:
- note added: "NOTE: The RGBx pins are open-drain and not push-pull!"
- note removed: "NOTE: The RGBx pins are open-drain!"
- moved on the sheet: R1013

Commit message: x65-sbc: pcb done
Parts:
- renumbered D402 to D1003, R415 to R1014, R415 to R1015
Connections:
- no-connect marks 4 -> 7
Other:
- note added: ""SDC ACTIVITY""
Changed lines of the file:
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@@
   (title_block
     (title "X65-SBC")
-    (date "2023-12-29")
+    (date "2024-01-10")
     (rev "revA1")
     (company "FOR X65.EU DESIGNED BY JSYKORA.INFO")
@@
   )
   (no_connect (at 56.515 90.805))
+  (no_connect (at 191.77 62.23))
+  (no_connect (at 191.77 54.61))
   (no_connect (at 56.515 88.265))
+  (no_connect (at 191.77 52.07))
   (no_connect (at 56.515 85.725))
   (no_connect (at 116.84 55.245))
@@
   )
   (text "package QFN-48" (at 59.69 100.965 0)
+    (effects (font (size 1.27 1.27)) (justify left bottom))
+  )
+  (text "\"SDC ACTIVITY\"" (at 137.16 153.67 0)
     (effects (font (size 1.27 1.27)) (justify left bottom))
   )
@@
   )
   (symbol (lib_id "Device:R") (at 193.675 127.635 0) (mirror y) (unit 1)
-    (in_bom yes) (on_board yes) (dnp no) (fields_autoplaced)
-    (property "Reference" "R1010" (at 196.215 126.3649 0)
+    (in_bom yes) (on_board yes) (dnp no)
+    (property "Reference" "R1010" (at 186.055 125.73 0)
       (effects (font (size 1.27 1.27)) (justify right))
     )
-    (property "Value" "10k" (at 196.215 128.9049 0)
+    (property "Value" "10k" (at 186.055 128.27 0)
       (effects (font (size 1.27 1.27)) (justify right))
     )
@@
   (symbol (lib_id "Device:LED") (at 143.51 146.685 0) (unit 1)
     (in_bom yes) (on_board yes) (dnp no)
-    (property "Reference" "D402" (at 141.9225 139.7 0)
+    (property "Reference" "D1003" (at 141.9225 139.7 0)
       (effects (font (size 1.27 1.27)))
     )
@@
     (instances
       (project "x65-sbc-revA1"
-        (path "/85750bea-43a1-4629-9575-611e72af7f9f/a0a926f8-222f-4537-8c1a-4e84db3f94e8"
-          (reference "D402") (unit 1)
-        )
         (path "/85750bea-43a1-4629-9575-611e72af7f9f/2791830c-aa1e-450d-95c0-111f156ac8ab"
           (reference "D1003") (unit 1)
@@
   (symbol (lib_id "Device:R") (at 128.27 138.43 90) (unit 1)
     (in_bom no) (on_board yes) (dnp yes)
-    (property "Reference" "R415" (at 128.27 135.89 90)
+    (property "Reference" "R1015" (at 128.27 135.89 90)
       (effects (font (size 1.27 1.27)))
     )
@@
     (instances
       (project "x65-sbc-revA1"
-        (path "/85750bea-43a1-4629-9575-611e72af7f9f/a0a926f8-222f-4537-8c1a-4e84db3f94e8"
-          (reference "R415") (unit 1)
-        )
         (path "/85750bea-43a1-4629-9575-611e72af7f9f/2791830c-aa1e-450d-95c0-111f156ac8ab"
           (reference "R1015") (unit 1)
@@
   (symbol (lib_id "Device:R") (at 128.27 146.685 90) (unit 1)
     (in_bom yes) (on_board yes) (dnp no)
-    (property "Reference" "R415" (at 128.27 144.145 90)
+    (property "Reference" "R1014" (at 128.27 144.145 90)
       (effects (font (size 1.27 1.27)))
     )
@@
     (instances
       (project "x65-sbc-revA1"
-        (path "/85750bea-43a1-4629-9575-611e72af7f9f/a0a926f8-222f-4537-8c1a-4e84db3f94e8"
-          (reference "R415") (unit 1)
-        )
         (path "/85750bea-43a1-4629-9575-611e72af7f9f/2791830c-aa1e-450d-95c0-111f156ac8ab"
           (reference "R1014") (unit 1)
