File: pcb/x65-sbc-revA1/11-sndout.kicad_sch (KiCad schematic)
At the start: 30 parts, among them J1101 PINS 1x2, J1104 JC-128, U1101 WM8524CGEDT, U1102 LM4890MX

Commit message: pcb sbc: more pcb work
Parts:
- added R1113: 0R, Resistor_SMD:R_0603_1608Metric_Pad0.98x0.95mm_HandSolder, symbol Device:R
Connections:
- net MONOMIX: now reaches R1101.1, R1102.2, R1103.2, R1104.2, R1111.2
- net MONOMIX: now also R1113.1; no longer C1101.1
- new net: C1101.1, R1113.2
Other:
- moved on the sheet: R1101, R1102, R1103, R1104, R1111

Commit message: x65-sbc: pcb done
Parts:
- removed C1110: 1u, Capacitor_SMD:C_0603_1608Metric_Pad1.08x0.95mm_HandSolder, symbol Device:C_Small
- R1101: now fitted
Connections:
- net GND: no longer J1104.G
Other:
- moved on the sheet: C1112
Changed lines of the file:
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@@
   (title_block
     (title "X65-SBC")
-    (date "2023-12-29")
+    (date "2024-01-10")
     (rev "revA1")
     (company "FOR X65.EU DESIGNED BY JSYKORA.INFO")
@@
     (stroke (width 0) (type default))
   )
-  (wire (pts (xy 111.76 120.65) (xy 113.03 120.65))
-    (stroke (width 0) (type default))
-  )
   (wire (pts (xy 91.44 69.85) (xy 91.44 71.12))
     (stroke (width 0) (type default))
@@
   )
   (symbol (lib_id "Device:R") (at 54.61 135.89 0) (unit 1)
-    (in_bom yes) (on_board yes) (dnp yes) (fields_autoplaced)
+    (in_bom yes) (on_board yes) (dnp no) (fields_autoplaced)
     (property "Reference" "R1101" (at 57.15 135.255 0)
       (effects (font (size 1.27 1.27)) (justify left))
@@
     )
   )
-  (symbol (lib_id "power:+5V") (at 140.97 154.305 0) (unit 1)
-    (in_bom yes) (on_board yes) (dnp no)
-    (property "Reference" "#PWR01114" (at 140.97 158.115 0)
-      (effects (font (size 1.27 1.27)) hide)
-    )
-    (property "Value" "+5V" (at 140.97 150.495 0)
-      (effects (font (size 1.27 1.27)))
-    )
-    (property "Footprint" "" (at 140.97 154.305 0)
-      (effects (font (size 1.27 1.27)) hide)
-    )
-    (property "Datasheet" "" (at 140.97 154.305 0)
-      (effects (font (size 1.27 1.27)) hide)
-    )
-    (pin "1")
-    (instances
-      (project "x65-sbc-revA1"
-        (path "/85750bea-43a1-4629-9575-611e72af7f9f/9182bec6-3ccd-452b-960c-9e4105d1fed5"
-          (reference "#PWR01114") (unit 1)
-        )
-      )
-      (project "openX65-vabo"
-        (path "/b8085944-4b3e-4781-a52b-94fe64f9a100/6ce180f3-0f22-4131-bc51-4e74cc150d15"
-          (reference "#PWR0720") (unit 1)
-        )
-      )
-    )
-  )
   (symbol (lib_id "Device:R_Potentiometer_Trim") (at 113.665 101.6 90) (unit 1)
     (in_bom yes) (on_board yes) (dnp no)
@@
     )
   )
-  (symbol (lib_id "power:GND") (at 113.03 120.65 90) (mirror x) (unit 1)
+  (symbol (lib_id "power:GND") (at 114.3 120.65 90) (mirror x) (unit 1)
     (in_bom yes) (on_board yes) (dnp no)
-    (property "Reference" "#PWR01112" (at 119.38 120.65 0)
+    (property "Reference" "#PWR01112" (at 120.65 120.65 0)
       (effects (font (size 1.27 1.27)) hide)
     )
-    (property "Value" "GND" (at 117.4242 120.777 0)
+    (property "Value" "GND" (at 118.6942 120.777 0)
       (effects (font (size 1.27 1.27)))
     )
-    (property "Footprint" "" (at 113.03 120.65 0)
+    (property "Footprint" "" (at 114.3 120.65 0)
       (effects (font (size 1.27 1.27)) hide)
     )
-    (property "Datasheet" "" (at 113.03 120.65 0)
+    (property "Datasheet" "" (at 114.3 120.65 0)
       (effects (font (size 1.27 1.27)) hide)
     )
@@
     )
   )
-  (symbol (lib_id "power:GND") (at 232.41 63.5 0) (mirror y) (unit 1)
-    (in_bom yes) (on_board yes) (dnp no)
-    (property "Reference" "#PWR01103" (at 232.41 69.85 0)
-      (effects (font (size 1.27 1.27)) hide)
-    )
-    (property "Value" "GND" (at 232.283 67.8942 0)
-      (effects (font (size 1.27 1.27)))
-    )
-    (property "Footprint" "" (at 232.41 63.5 0)
-      (effects (font (size 1.27 1.27)) hide)
-    )
-    (property "Datasheet" "" (at 232.41 63.5 0)
-      (effects (font (size 1.27 1.27)) hide)
-    )
-    (pin "1")
-    (instances
-      (project "x65-sbc-revA1"
-        (path "/85750bea-43a1-4629-9575-611e72af7f9f/9182bec6-3ccd-452b-960c-9e4105d1fed5"
-          (reference "#PWR01103") (unit 1)
-        )
-      )
-      (project "openX65-vabo"
-        (path "/b8085944-4b3e-4781-a52b-94fe64f9a100/6ce180f3-0f22-4131-bc51-4e74cc150d15"
-          (reference "#PWR0705") (unit 1)
-        )
-      )
-    )
-  )
   (symbol (lib_id "power:GND") (at 227.33 48.26 270) (mirror x) (unit 1)
     (in_bom yes) (on_board yes) (dnp no)
@@
     )
   )
-  (symbol (lib_id "Device:C") (at 140.97 158.115 180) (unit 1)
+  (symbol (lib_id "Device:C") (at 110.49 120.65 270) (unit 1)
     (in_bom yes) (on_board yes) (dnp no)
-    (property "Reference" "C1112" (at 135.89 157.48 0)
+    (property "Reference" "C1112" (at 112.395 114.935 90)
       (effects (font (size 1.27 1.27)))
     )
-    (property "Value" "22u/16V" (at 133.985 160.02 0)
+    (property "Value" "22u/16V" (at 113.665 116.84 90)
       (effects (font (size 1.27 1.27)))
     )
-    (property "Footprint" "Capacitor_SMD:C_0805_2012Metric_Pad1.18x1.45mm_HandSolder" (at 140.0048 154.305 0)
+    (property "Footprint" "Capacitor_SMD:C_0805_2012Metric_Pad1.18x1.45mm_HandSolder" (at 106.68 121.6152 0)
       (effects (font (size 1.27 1.27)) hide)
     )
-    (property "Datasheet" "~" (at 140.97 158.115 0)
+    (property "Datasheet" "~" (at 110.49 120.65 0)
       (effects (font (size 1.27 1.27)) hide)
     )
@@
     )
   )
-  (symbol (lib_id "Device:C_Small") (at 109.22 120.65 90) (unit 1)
-    (in_bom yes) (on_board yes) (dnp no)
-    (property "Reference" "C1110" (at 108.0516 118.3132 0)
-      (effects (font (size 1.27 1.27)) (justify left))
-    )
-    (property "Value" "1u" (at 110.363 118.3132 0)
-      (effects (font (size 1.27 1.27)) (justify left))
-    )
-    (property "Footprint" "Capacitor_SMD:C_0603_1608Metric_Pad1.08x0.95mm_HandSolder" (at 109.22 120.65 0)
-      (effects (font (size 1.27 1.27)) hide)
-    )
-    (property "Datasheet" "~" (at 109.22 120.65 0)
-      (effects (font (size 1.27 1.27)) hide)
-    )
-    (pin "1")
-    (pin "2")
-    (instances
-      (project "x65-sbc-revA1"
-        (path "/85750bea-43a1-4629-9575-611e72af7f9f/9182bec6-3ccd-452b-960c-9e4105d1fed5"
-          (reference "C1110") (unit 1)
-        )
-      )
-      (project "openX65-vabo"
-        (path "/b8085944-4b3e-4781-a52b-94fe64f9a100/6ce180f3-0f22-4131-bc51-4e74cc150d15"
-          (reference "C711") (unit 1)
-        )
-      )
-    )
-  )
-  (symbol (lib_id "power:GND") (at 140.97 161.925 0) (mirror y) (unit 1)
-    (in_bom yes) (on_board yes) (dnp no)
-    (property "Reference" "#PWR01115" (at 140.97 168.275 0)
-      (effects (font (size 1.27 1.27)) hide)
-    )
-    (property "Value" "GND" (at 140.843 166.3192 0)
-      (effects (font (size 1.27 1.27)))
-    )
-    (property "Footprint" "" (at 140.97 161.925 0)
-      (effects (font (size 1.27 1.27)) hide)
-    )
-    (property "Datasheet" "" (at 140.97 161.925 0)
-      (effects (font (size 1.27 1.27)) hide)
-    )
-    (pin "1")
-    (instances
-      (project "x65-sbc-revA1"
-        (path "/85750bea-43a1-4629-9575-611e72af7f9f/9182bec6-3ccd-452b-960c-9e4105d1fed5"
-          (reference "#PWR01115") (unit 1)
-        )
-      )
-      (project "openX65-vabo"
-        (path "/b8085944-4b3e-4781-a52b-94fe64f9a100/6ce180f3-0f22-4131-bc51-4e74cc150d15"
-          (reference "#PWR0721") (unit 1)
-        )
-      )
-    )
-  )
   (symbol (lib_id "Device:R") (at 45.72 128.27 90) (unit 1)
     (in_bom yes) (on_board yes) (dnp no)
@@
       (effects (font (size 1.27 1.27)) hide)
     )
-    (pin "G")
     (pin "R")
     (pin "RN")
