File: pcb/x65-sbc-revA1/12-ethernet.kicad_sch (KiCad schematic)
At the start: 40 parts, among them J1201 RJMG1BD3B8K1ANR, U1201 W6100L, U1203 24AA025E48T-I/OT

Commit message: pcb sbc: more pcb work
Parts:
- removed C1203: 22u/16V, Capacitor_SMD:C_0805_2012Metric_Pad1.18x1.45mm_HandSolder, symbol Device:C
- removed C1207, C1211, C1212: 1u, Capacitor_SMD:C_0603_1608Metric_Pad1.08x0.95mm_HandSolder, symbol Device:C_Small
Connections:
- net ESYSCLK renamed 25MHz
Other:
- note added: "EEPROM 24AA025E48 I2C DEVICE ADDRESS (8b=shifted) = 0b1010_000W = 0xA0, that is 7-bit address = 0x28"
- note removed: "EEPROM 24AA025E48 I2C DEVICE ADDRESS (8b=shifted) = 0b1010_000W = 0xA0"
