File: pcb/x65-sbc-revA1/03-nora_fpga.kicad_sch (KiCad schematic)
At the start: 38 parts, among them Q301 BSS138, SW401 PTS645VM13SMTR92 LFS, U301 ICE40HX4K-TQ144, U302 W25Q128JVS, U303 IS25WP256D-xM, W25Q512JVFIQ, X301 SG5032CAN 12.000000M-TJGA0

Commit message: pcb sbc: more pcb work
Connections:
- net UART_CTS: now also U301.113 (IOT_170); no longer U301.112 (IOT_169)
- net UART_RTS: now also U301.112 (IOT_169); no longer U301.113 (IOT_170)
- net DIPLED0: now reaches U301.125 (IOT_192)
- net DIPLED1: now reaches U301.137 (IOT_215)
Other:
- note added: "package: SOIC-8 5.23x5.23mm 208mil (up to 128Mbit) or SOIC-8 3.9x4.9mm 150mil (up to 16Mbit)"
- note removed: "package: SOIC-8 5.23x5.23mm 208mil (up to 128Mbit) AND SOIC-8 3.9x4.9mm 150mil (up to 16Mbit)"
Changed lines of the file:
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@@
     (stroke (width 0) (type default))
   )
-  (text "package: SOIC-8 5.23x5.23mm 208mil (up to 128Mbit)\nAND SOIC-8 3.9x4.9mm 150mil (up to 16Mbit) "
+  (text "package: SOIC-8 5.23x5.23mm 208mil (up to 128Mbit)\n    or SOIC-8 3.9x4.9mm 150mil (up to 16Mbit) "
     (at 77.47 186.69 0)
     (effects (font (size 1.27 1.27)) (justify left bottom))
@@
     )
   )
-  (global_label "UART_RTS" (shape input) (at 252.73 41.91 180) (fields_autoplaced)
-    (effects (font (size 1.27 1.27)) (justify right))
-    (property "Intersheetrefs" "${INTERSHEET_REFS}" (at 241.2455 41.8306 0)
+  (global_label "UART_RTS" (shape output) (at 252.73 39.37 180) (fields_autoplaced)
+    (effects (font (size 1.27 1.27)) (justify right))
+    (property "Intersheetrefs" "${INTERSHEET_REFS}" (at 240.6734 39.37 0)
       (effects (font (size 1.27 1.27)) (justify right) hide)
     )
@@
     )
   )
-  (global_label "UART_CTS" (shape output) (at 252.73 39.37 180) (fields_autoplaced)
-    (effects (font (size 1.27 1.27)) (justify right))
-    (property "Intersheetrefs" "${INTERSHEET_REFS}" (at 241.2455 39.2906 0)
+  (global_label "UART_CTS" (shape input) (at 252.73 41.91 180) (fields_autoplaced)
+    (effects (font (size 1.27 1.27)) (justify right))
+    (property "Intersheetrefs" "${INTERSHEET_REFS}" (at 240.6734 41.91 0)
       (effects (font (size 1.27 1.27)) (justify right) hide)
     )
@@
       (effects (font (size 1.27 1.27)) (justify right) hide)
     )
+  )
+  (global_label "DIPLED0" (shape bidirectional) (at 252.73 69.85 180) (fields_autoplaced)
+    (effects (font (size 1.27 1.27)) (justify right))
+    (property "Intersheetrefs" "${INTERSHEET_REFS}" (at 240.8321 69.85 0)
+      (effects (font (size 1.27 1.27)) (justify right) hide)
+    )
+  )
+  (global_label "DIPLED1" (shape bidirectional) (at 252.73 87.63 180) (fields_autoplaced)
+    (effects (font (size 1.27 1.27)) (justify right))
+    (property "Intersheetrefs" "${INTERSHEET_REFS}" (at 240.8321 87.63 0)
+      (effects (font (size 1.27 1.27)) (justify right) hide)
+    )

Commit message: x65-sbc: pcb done
Parts:
- renumbered SW401 to SW301
Connections:
- net NESCLOCK: now also U301.135 (IOT_213); no longer U301.134 (IOT_212)
- net NESDATA0: now also U301.130 (IOT_206); no longer U301.136 (IOT_214)
- net NESDATA1: now also U301.134 (IOT_212); no longer U301.135 (IOT_213)
- net NESLATCH: now also U301.136 (IOT_214); no longer U301.130 (IOT_206)
- net ~{UE_CS3}: now also U301.95 (IOR_144); no longer U301.81 (IOR_117)
- net ~{UE_IRQ}: now also U301.81 (IOR_117); no longer U301.95 (IOR_144)
Changed lines of the file:
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@@
   (title_block
     (title "X65-SBC")
-    (date "2023-12-29")
+    (date "2024-01-10")
     (rev "revA1")
     (company "FOR X65.EU DESIGNED BY JSYKORA.INFO")
@@
   (no_connect (at 194.31 74.93))
   (no_connect (at 140.335 137.16))
-  (bus_entry (at 237.49 92.71) (size 2.54 2.54)
+  (bus_entry (at 234.315 92.71) (size 2.54 2.54)
     (stroke (width 0) (type default))
   )
@@
     (stroke (width 0) (type default))
   )
-  (bus_entry (at 237.49 90.17) (size 2.54 2.54)
-    (stroke (width 0) (type default))
-  )
-  (bus_entry (at 237.49 87.63) (size 2.54 2.54)
+  (bus_entry (at 234.315 90.17) (size 2.54 2.54)
+    (stroke (width 0) (type default))
+  )
+  (bus_entry (at 234.315 87.63) (size 2.54 2.54)
     (stroke (width 0) (type default))
   )
@@
     (stroke (width 0) (type default))
   )
-  (bus (pts (xy 234.95 85.09) (xy 237.49 85.09))
+  (bus (pts (xy 231.775 85.09) (xy 234.315 85.09))
     (stroke (width 0) (type default))
   )
@@
     (stroke (width 0) (type default))
   )
-  (bus (pts (xy 237.49 87.63) (xy 237.49 90.17))
+  (bus (pts (xy 234.315 87.63) (xy 234.315 90.17))
     (stroke (width 0) (type default))
   )
@@
     (stroke (width 0) (type default))
   )
-  (wire (pts (xy 240.03 90.17) (xy 252.73 90.17))
+  (wire (pts (xy 236.855 90.17) (xy 252.73 90.17))
     (stroke (width 0) (type default))
   )
@@
     (stroke (width 0) (type default))
   )
-  (bus (pts (xy 237.49 87.63) (xy 237.49 85.09))
+  (bus (pts (xy 234.315 87.63) (xy 234.315 85.09))
     (stroke (width 0) (type default))
   )
@@
     (stroke (width 0) (type default))
   )
-  (wire (pts (xy 240.03 92.71) (xy 252.73 92.71))
-    (stroke (width 0) (type default))
-  )
   (bus (pts (xy 139.7 30.48) (xy 139.7 39.37))
     (stroke (width 0) (type default))
@@
     (stroke (width 0) (type default))
   )
-  (bus (pts (xy 237.49 92.71) (xy 237.49 90.17))
+  (bus (pts (xy 234.315 92.71) (xy 234.315 90.17))
     (stroke (width 0) (type default))
   )
@@
     (stroke (width 0) (type default))
   )
-  (wire (pts (xy 240.03 95.25) (xy 252.73 95.25))
-    (stroke (width 0) (type default))
-  )
   (bus (pts (xy 45.72 105.41) (xy 45.72 107.95))
     (stroke (width 0) (type default))
@@
     (stroke (width 0) (type default))
   )
+  (wire (pts (xy 236.855 95.25) (xy 252.73 95.25))
+    (stroke (width 0) (type default))
+  )
   (wire (pts (xy 236.22 123.19) (xy 245.11 123.19))
     (stroke (width 0) (type default))
@@
   )
   (wire (pts (xy 189.23 67.31) (xy 189.23 71.12))
+    (stroke (width 0) (type default))
+  )
+  (wire (pts (xy 236.855 92.71) (xy 252.73 92.71))
     (stroke (width 0) (type default))
   )
@@
     (effects (font (size 1.27 1.27)) (justify left bottom))
   )
-  (label "A13" (at 241.3 92.71 0) (fields_autoplaced)
+  (label "A13" (at 237.49 92.71 0) (fields_autoplaced)
     (effects (font (size 1.27 1.27)) (justify left bottom))
   )
@@
     (effects (font (size 1.27 1.27)) (justify left bottom))
   )
-  (label "A12" (at 241.3 90.17 0) (fields_autoplaced)
+  (label "A12" (at 237.49 90.17 0) (fields_autoplaced)
     (effects (font (size 1.27 1.27)) (justify left bottom))
   )
@@
     (effects (font (size 1.27 1.27)) (justify left bottom))
   )
-  (label "A14" (at 241.3 95.25 0) (fields_autoplaced)
+  (label "A14" (at 237.49 95.25 0) (fields_autoplaced)
     (effects (font (size 1.27 1.27)) (justify left bottom))
   )
@@
     (effects (font (size 1.27 1.27)) (justify left bottom))
   )
-  (global_label "A[0..20]" (shape bidirectional) (at 234.95 85.09 180) (fields_autoplaced)
-    (effects (font (size 1.27 1.27)) (justify right))
-    (property "Intersheetrefs" "${INTERSHEET_REFS}" (at 224.9169 85.0106 0)
+  (global_label "A[0..20]" (shape bidirectional) (at 231.775 85.09 180) (fields_autoplaced)
+    (effects (font (size 1.27 1.27)) (justify right))
+    (property "Intersheetrefs" "${INTERSHEET_REFS}" (at 221.7419 85.0106 0)
       (effects (font (size 1.27 1.27)) (justify right) hide)
     )
@@
     )
   )
-  (global_label "NESCLOCK" (shape output) (at 252.73 80.01 180) (fields_autoplaced)
-    (effects (font (size 1.27 1.27)) (justify right))
-    (property "Intersheetrefs" "${INTERSHEET_REFS}" (at 240.4593 80.0894 0)
+  (global_label "NESCLOCK" (shape output) (at 252.73 82.55 180) (fields_autoplaced)
+    (effects (font (size 1.27 1.27)) (justify right))
+    (property "Intersheetrefs" "${INTERSHEET_REFS}" (at 240.4593 82.6294 0)
       (effects (font (size 1.27 1.27)) (justify right) hide)
     )
@@
     )
   )
-  (global_label "~{UE_CS3}" (shape output) (at 152.4 54.61 180) (fields_autoplaced)
-    (effects (font (size 1.27 1.27)) (justify right))
-    (property "Intersheetrefs" "${INTERSHEET_REFS}" (at 142.3581 54.61 0)
+  (global_label "~{UE_CS3}" (shape output) (at 152.4 82.55 180) (fields_autoplaced)
+    (effects (font (size 1.27 1.27)) (justify right))
+    (property "Intersheetrefs" "${INTERSHEET_REFS}" (at 142.3581 82.55 0)
       (effects (font (size 1.27 1.27)) (justify right) hide)
     )
@@
     )
   )
-  (global_label "~{UE_IRQ}" (shape input) (at 152.4 82.55 180) (fields_autoplaced)
-    (effects (font (size 1.27 1.27)) (justify right))
-    (property "Intersheetrefs" "${INTERSHEET_REFS}" (at 142.8418 82.55 0)
+  (global_label "~{UE_IRQ}" (shape input) (at 152.4 54.61 180) (fields_autoplaced)
+    (effects (font (size 1.27 1.27)) (justify right))
+    (property "Intersheetrefs" "${INTERSHEET_REFS}" (at 142.8418 54.61 0)
       (effects (font (size 1.27 1.27)) (justify right) hide)
     )
@@
     )
   )
-  (global_label "NESDATA0" (shape input) (at 252.73 85.09 180) (fields_autoplaced)
-    (effects (font (size 1.27 1.27)) (justify right))
-    (property "Intersheetrefs" "${INTERSHEET_REFS}" (at 241.0036 85.0106 0)
+  (global_label "NESDATA0" (shape input) (at 252.73 77.47 180) (fields_autoplaced)
+    (effects (font (size 1.27 1.27)) (justify right))
+    (property "Intersheetrefs" "${INTERSHEET_REFS}" (at 241.0036 77.3906 0)
       (effects (font (size 1.27 1.27)) (justify right) hide)
     )
@@
     )
   )
-  (global_label "NESDATA1" (shape input) (at 252.73 82.55 180) (fields_autoplaced)
-    (effects (font (size 1.27 1.27)) (justify right))
-    (property "Intersheetrefs" "${INTERSHEET_REFS}" (at 241.0036 82.6294 0)
+  (global_label "NESDATA1" (shape input) (at 252.73 80.01 180) (fields_autoplaced)
+    (effects (font (size 1.27 1.27)) (justify right))
+    (property "Intersheetrefs" "${INTERSHEET_REFS}" (at 241.0036 80.0894 0)
       (effects (font (size 1.27 1.27)) (justify right) hide)
     )
@@
     )
   )
-  (global_label "NESLATCH" (shape output) (at 252.73 77.47 180) (fields_autoplaced)
-    (effects (font (size 1.27 1.27)) (justify right))
-    (property "Intersheetrefs" "${INTERSHEET_REFS}" (at 240.9431 77.5494 0)
+  (global_label "NESLATCH" (shape output) (at 252.73 85.09 180) (fields_autoplaced)
+    (effects (font (size 1.27 1.27)) (justify right))
+    (property "Intersheetrefs" "${INTERSHEET_REFS}" (at 240.9431 85.1694 0)
       (effects (font (size 1.27 1.27)) (justify right) hide)
     )
@@
   (symbol (lib_id "vera-module:SW_Push_SH") (at 193.675 107.95 90) (unit 1)
     (in_bom yes) (on_board yes) (dnp no)
-    (property "Reference" "SW401" (at 185.42 107.95 0)
+    (property "Reference" "SW301" (at 185.42 107.95 0)
       (effects (font (size 1.27 1.27)))
     )
@@
     (instances
       (project "x65-sbc-revA1"
-        (path "/85750bea-43a1-4629-9575-611e72af7f9f/00150742-fc5e-4d8a-b33f-e79b4d66582a"
-          (reference "SW401") (unit 1)
-        )
         (path "/85750bea-43a1-4629-9575-611e72af7f9f/17c238d7-f888-4cc2-8790-8144029e69c2"
           (reference "SW301") (unit 1)

Commit message: pcb/scm x65-sbc update
Parts:
- SW301: footprint switches:PTS645VM13SMTR92 LFS -> x65_footprints:PTS645VM13SMTR92 LFS
Changed lines of the file:
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@@
       (effects (font (size 1.27 1.27)))
     )
-    (property "Footprint" "switches:PTS645VM13SMTR92 LFS" (at 188.595 107.95 0)
+    (property "Footprint" "x65_footprints:PTS645VM13SMTR92 LFS" (at 188.595 107.95 0)
       (effects (font (size 1.27 1.27)) hide)
     )
