File: pcb/x65-sbc-revB1/x65-sbc-revB1.kicad_pcb (KiCad board)
At the start: 4 copper layers, 100 x 180 mm, 344 parts, among them J1101 PINS 1x2, J1104 JC-128, J1201 RJMG1BD3B8K1ANR, J403 SNES_Controller_Conn, J404 SNES_Controller_Conn, J501 USB4085-GF-A, J601 IDC PINS 2x10p 2,54mm, J603 DS1013-10RSIB CONNFLY, J605 TE 5749180-1, J606 TE 5749180-1, J701 Conn_01x02, J702 Conn_01x01, J703 Conn_01x01, J704 Conn_01x01, J801 ICD15S13E4GV00LF, J901 DM1AA-SF-PEJ, Q1001 BSS138, Q301 BSS138, Q601 BSS138, Q602 BSS138, Q603 BSS138, Q604 BSS138, Q801 BSS138, SW301 PTS645VM13SMTR92 LFS, SW401 SW_DIP_x02 TE 1825058-1, U1001 ICE40UP5K-SG48ITR50, U1002 74CBTLV3126PW,118, U1003 W25Q16JVSNIQ, U1101 WM8524CGEDT, U1102 LM4890MX, U1201 W6100L, U1203 24AA025E48T-I/OT, U201 W65C816S6TQG-14, U202 IS61WV20488FBLL-10TLI, U301 ICE40HX4K-TQ144, U302 W25Q128JVS, U303 IS25WP256D-xM, W25Q512JVFIQ, U401 74LVC2G17DBVR, U402 MCP7940N-xSN, U403 74LVC2G17DBVR, U501 SN74LVC1G08DBVR, U503 74CBTLV3126PW,118, U504 FT2232HL, U701 MP2149GJ, U801 ICE40UP5K-SG48ITR50, U901 74CBTLV3126PW,118, U902 74CBTLV3126PW,118, U903 74AHC00PW, U904 W25Q16JVSNIQ, X301 SG5032CAN 12.000000M-TJGA0, X801 SG5032CAN_25.000000M-TJGA3, Y402 CM8V-T1A-32.768kHz-9pF-20PPM-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

Commit message: update sbc-revB1
Parts:
- removed the G*** at (75.0, 194.0)
- added G***: LOGO, x65_footprints:qrlink-x65github, B.Cu at (74.6, 193.7)
