File: pcb/x65-sbc-revB1/x65-sbc-revB1.kicad_sch (KiCad schematic)
At the start: 9 parts

Commit message: update sbc-revB1
Other:
- note added: "X65 SBC rev.B1"
- note removed: "X65 SBC rev.A1"
Changed lines of the file:
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@@
     (effects (font (size 5 5)) (justify left bottom))
   )
-  (text "X65 SBC rev.A1" (at 22.86 31.75 0)
+  (text "X65 SBC rev.B1" (at 22.86 31.75 0)
     (effects (font (size 10 10) (thickness 2) bold) (justify left bottom))
   )
